File: KontollerTKDNTinggi/KontollerTKDNTinggi.kicad_sch (KiCad schematic)
At the start: 107 parts, among them J1 AH_Conn, J10 Ready, J16 CtrlON, J2 AL_Conn, J3 BH_Conn, J4 BL_Conn, J5 CH_Conn, J6 CL_Conn, J7 SignalA, J8 SignalB, J9 SignalB, Q1 AO3401A, Q10 A03400, Q11 A03400, Q12 AO3400, Q13 AO3400, Q14 AO3400, Q15 AO3401, Q4 AO3401, Q5 AO3401, Q6 AO3401, Q7 AO3401, Q9 A03400, U13 LM5161PWP, U14 LM2596S-5, U15 INA241A2xD, U16 INA241A2xD, U17 INA241A2xD

Commit message: ngetesdoang
Parts:
- removed R95: 1k1, symbol Device:R
Changed lines of the file:
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@@
 	)
 	(junction
-		(at 262.89 130.81)
-		(diameter 0)
-		(color 0 0 0 0)
-	)
-	(junction
 		(at 85.09 167.64)
 		(diameter 0)
@@
 	(wire
 		(pts
-			(xy 257.81 130.81) (xy 262.89 130.81)
-		)
-		(stroke
-			(width 0)
-			(type default)
-		)
-	)
-	(wire
-		(pts
 			(xy 351.79 135.89) (xy 345.44 135.89)
 		)
@@
 	(wire
 		(pts
-			(xy 262.89 130.81) (xy 267.97 130.81)
+			(xy 257.81 130.81) (xy 267.97 130.81)
 		)
 		(stroke
@@
 					(unit 1)
 				)
-			)
-		)
-	)
-	(symbol
-		(lib_id "Device:R")
-		(at 262.89 127 0)
-		(mirror y)
-		(unit 1)
-		(exclude_from_sim no)
-		(in_bom yes)
-		(on_board yes)
-		(dnp no)
-		(property "Reference" "R95"
-			(at 262.89 127 90)
-			(effects
-				(font
-					(size 1.27 1.27)
-				)
-			)
-		)
-		(property "Value" "1k1"
-			(at 265.43 127 90)
-			(effects
-				(font
-					(size 1.27 1.27)
-				)
-			)
-		)
-		(property "Footprint" ""
-			(at 264.668 127 90)
-			(effects
-				(font
-					(size 1.27 1.27)
-				)
-				(hide yes)
-			)
-		)
-		(property "Datasheet" "~"
-			(at 262.89 127 0)
-			(effects
-				(font
-					(size 1.27 1.27)
-				)
-				(hide yes)
-			)
-		)
-		(property "Description" "Resistor"
-			(at 262.89 127 0)
-			(effects
-				(font
-					(size 1.27 1.27)
-				)
-				(hide yes)
-			)
-		)
-		(pin "1"
-		)
-		(pin "2"
-		)
-		(instances
-			(project "KontollerTKDNTinggi"
-				(path "/a2f3e1cd-dd27-43de-a976-b374057486e7"
-					(reference "R95")
-					(unit 1)
-				)

Commit message: real
Parts:
- added R95: 1k1, symbol Device:R
Connections:
- net GND: now also R95.1
- net at R100.2, R89.1, U9.1 (+In1): now also R95.2
Changed lines of the file:
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@@
 	)
 	(junction
+		(at 262.89 130.81)
+		(diameter 0)
+		(color 0 0 0 0)
+	)
+	(junction
 		(at 85.09 167.64)
 		(diameter 0)
@@
 	(wire
 		(pts
+			(xy 257.81 130.81) (xy 262.89 130.81)
+		)
+		(stroke
+			(width 0)
+			(type default)
+		)
+	)
+	(wire
+		(pts
 			(xy 351.79 135.89) (xy 345.44 135.89)
 		)
@@
 	(wire
 		(pts
-			(xy 257.81 130.81) (xy 267.97 130.81)
+			(xy 262.89 130.81) (xy 267.97 130.81)
 		)
 		(stroke
@@
 					(unit 1)
 				)
+			)
+		)
+	)
+	(symbol
+		(lib_id "Device:R")
+		(at 262.89 127 0)
+		(mirror y)
+		(unit 1)
+		(exclude_from_sim no)
+		(in_bom yes)
+		(on_board yes)
+		(dnp no)
+		(property "Reference" "R95"
+			(at 262.89 127 90)
+			(effects
+				(font
+					(size 1.27 1.27)
+				)
+			)
+		)
+		(property "Value" "1k1"
+			(at 265.43 127 90)
+			(effects
+				(font
+					(size 1.27 1.27)
+				)
+			)
+		)
+		(property "Footprint" ""
+			(at 264.668 127 90)
+			(effects
+				(font
+					(size 1.27 1.27)
+				)
+				(hide yes)
+			)
+		)
+		(property "Datasheet" "~"
+			(at 262.89 127 0)
+			(effects
+				(font
+					(size 1.27 1.27)
+				)
+				(hide yes)
+			)
+		)
+		(property "Description" "Resistor"
+			(at 262.89 127 0)
+			(effects
+				(font
+					(size 1.27 1.27)
+				)
+				(hide yes)
+			)
+		)
+		(pin "1"
+		)
+		(pin "2"
+		)
+		(instances
+			(project "KontollerTKDNTinggi"
+				(path "/a2f3e1cd-dd27-43de-a976-b374057486e7"
+					(reference "R95")
+					(unit 1)
+				)

Commit message: mynigga
Parts:
- removed R102: ref, symbol Device:R
Changed lines of the file:
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@@
-	)
-	(symbol
-		(lib_id "Device:R")
-		(at 278.13 162.56 270)
-		(unit 1)
-		(exclude_from_sim no)
-		(in_bom yes)
-		(on_board yes)
-		(dnp no)
-		(property "Reference" "R102"
-			(at 278.13 162.56 90)
-			(effects
-				(font
-					(size 1.27 1.27)
-				)
-			)
-		)
-		(property "Value" "ref"
-			(at 278.13 160.02 90)
-			(effects
-				(font
-					(size 1.27 1.27)
-				)
-			)
-		)
-		(property "Footprint" ""
-			(at 278.13 160.782 90)
-			(effects
-				(font
-					(size 1.27 1.27)
-				)
-				(hide yes)
-			)
-		)
-		(property "Datasheet" "~"
-			(at 278.13 162.56 0)
-			(effects
-				(font
-					(size 1.27 1.27)
-				)
-				(hide yes)
-			)
-		)
-		(property "Description" "Resistor"
-			(at 278.13 162.56 0)
-			(effects
-				(font
-					(size 1.27 1.27)
-				)
-				(hide yes)
-			)
-		)
-		(pin "1"
-		)
-		(pin "2"
-		)
-		(instances
-			(project "KontollerTKDNTinggi"
-				(path "/a2f3e1cd-dd27-43de-a976-b374057486e7"
-					(reference "R102")
-					(unit 1)
-				)
-			)
-		)
 	)
 	(symbol
