File: KontollerTKDNTinggi/KontollerTKDNTinggi.kicad_sch (KiCad schematic)
At the start: 105 parts, among them J1 AH_Conn, J10 Ready, J16 CtrlON, J2 AL_Conn, J3 BH_Conn, J4 BL_Conn, J5 CH_Conn, J6 CL_Conn, J7 SignalA, J8 SignalB, J9 SignalB, Q1 AO3401A, Q10 A03400, Q11 A03400, Q12 AO3400, Q13 AO3400, Q14 AO3400, Q15 AO3401, Q4 AO3401, Q5 AO3401, Q6 AO3401, Q7 AO3401, Q9 A03400, U13 LM5161PWP, U14 LM2596S-5, U15 INA241A2xD, U16 INA241A2xD, U17 INA241A2xD

Commit message: V2
Parts:
- added R96: 270, symbol Device:R
Connections:
- net OvercurrentB: now also R96.1
- net at R90.1, U10.1 (+In1): now also R96.2
Changed lines of the file:
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@@
+	(symbol
+		(lib_id "Device:R")
+		(at 278.13 162.56 270)
+		(unit 1)
+		(exclude_from_sim no)
+		(in_bom yes)
+		(on_board yes)
+		(dnp no)
+		(property "Reference" "R96"
+			(at 278.13 162.56 90)
+			(effects
+				(font
+					(size 1.27 1.27)
+				)
+			)
+		)
+		(property "Value" "270"
+			(at 278.13 160.02 90)
+			(effects
+				(font
+					(size 1.27 1.27)
+				)
+			)
+		)
+		(property "Footprint" ""
+			(at 278.13 160.782 90)
+			(effects
+				(font
+					(size 1.27 1.27)
+				)
+				(hide yes)
+			)
+		)
+		(property "Datasheet" "~"
+			(at 278.13 162.56 0)
+			(effects
+				(font
+					(size 1.27 1.27)
+				)
+				(hide yes)
+			)
+		)
+		(property "Description" "Resistor"
+			(at 278.13 162.56 0)
+			(effects
+				(font
+					(size 1.27 1.27)
+				)
+				(hide yes)
+			)
+		)
+		(pin "1"
+		)
+		(pin "2"
+		)
+		(instances
+			(project "KontollerTKDNTinggi"
+				(path "/a2f3e1cd-dd27-43de-a976-b374057486e7"
+					(reference "R96")
+					(unit 1)
+				)
+			)
+		)
+	)
 	(symbol
 		(lib_id "Device:R")

Commit message: 11Nov
Parts:
- added C23, C24, C25, C26: 2.2u, symbol Device:C
- added D1: LED RED, symbol Device:LED
- added J11: Ready, symbol Connector_Generic:Conn_01x02
- added J12: Throttle, symbol Connector_Generic:Conn_01x03
- added K2: IM06, customLib:RELAY8-TH_NON-LATCH_1-COIL, symbol Relay:IM06
- added Q16: PMOS, symbol Simulation_SPICE:PMOS
- added R54, R55: 1k, symbol Device:R
- added R56, R57: 51, symbol Device:R
- added R58, R59, R60: 120, symbol Device:R
- added U2: PC817, Package_DIP:DIP-4_W7.62mm, symbol Isolator:PC817
- added U3, U4: TJA1051T-3, Package_SO:SOIC-8_3.9x4.9mm_P1.27mm, symbol Interface_CAN_LIN:TJA1051T-3
Connections:
- net +12V: now also K2.8, Q16.1 (D), R57.2, U2.4
- net +3.3V: now also C24.2, C25.2, J12.3 (Pin_3), U3.5 (VIO), U4.5 (VIO)
- net +5V: now also U7.3 (5V), C23.2, C26.2, U3.3 (VCC), U4.3 (VCC)
- net ADC_15: now also U7.48 (A4)
- net CAN_RX: now also U3.4 (RXD)
- net CAN_TX: now also U3.1 (TXD)
- net Drive_Supply: now also D1.2 (A), Q16.3 (S)
- net Error: now also Q6.1 (D), K2.7, U2.1
- net GND: now also U7.33 (GND), C23.1, C24.1, C25.1, C26.1, J11.1 (Pin_1), J12.1 (Pin_1), R54.1, R55.1, R58.2, U3.2 (GND), U3.8 (S), U4.2 (GND), U4.8 (S)
- net at U7.1 (GND): now also U7.2 (GND), U7.30 (GND), U7.31 (GND), U7.35 (GND), U7.59 (GND)
- net CAN_RX1: now reaches U7.28 (B8)
- net CAN_RX1: now also U4.4 (RXD)
- net CAN_TX1: now reaches U7.29 (B9)
- net CAN_TX1: now also U4.1 (TXD)
- net DC_Current: now reaches U7.50 (A2)
- net Throttle_IN: now reaches U7.52 (A0)
- net Throttle_IN: now also J12.2 (Pin_2)
- new net: K2.5, R57.1
- new net: D1.1 (K), R58.1
- new net: R54.2, U2.2
- new net: Q16.2 (G), R56.2
- new net CAN_H: R59.1, R59.2, R60.1, R60.2, U3.6 (CANL), U3.7 (CANH), U4.6 (CANL), U4.7 (CANH)
- new net R2: K2.6, R55.2, R56.1, U2.3
- new net Reset: J11.2 (Pin_2), K2.1
Other:
- note added: "CAN_Transceiver"
- note added: "ERROR = LOW"
- note added: "RESET RELAY"
- moved on the sheet: H1, H2, H3, H4, J1, J10, J16, J2, J3, J4, J5, J6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

Commit message: ganticonnector
Parts:
- removed J10, J11: Ready, symbol Connector_Generic:Conn_01x02
- removed J12: Throttle, symbol Connector_Generic:Conn_01x03
- removed J16: CtrlON, Connector_Molex:Molex_Micro-Fit_3.0_43650-0200_1x02_P3.00mm_Horizontal, symbol Connector_Generic:Conn_01x02
- removed Q1: AO3401A, symbol Simulation_SPICE:PMOS
- removed Q10, Q11, Q9: A03400, symbol Simulation_SPICE:NMOS
- removed Q12, Q13, Q14: AO3400, symbol Simulation_SPICE:NMOS
- removed Q15, Q4, Q5, Q6, Q7: AO3401, symbol Simulation_SPICE:PMOS
- removed Q16: PMOS, symbol Simulation_SPICE:PMOS
- removed R44: 1k, symbol Device:R
- added C27: 100nF, Capacitor_SMD:C_0805_2012Metric_Pad1.18x1.45mm_HandSolder, symbol Device:C
- added C28: 47uF, Capacitor_SMD:CP_Elec_6.3x7.7, symbol Device:C_Polarized_US
- added D3: LED, LED_SMD:LED_0805_2012Metric_Pad1.15x1.40mm_HandSolder, symbol Device:LED
- added J13: 6473711-1, 6473711-1:TE_6473711-1, symbol 6473711-1:6473711-1
- added Q1, Q7: AO3401A, Package_TO_SOT_SMD:SOT-23, symbol Transistor_FET:AO3401A
- added Q10: HY19P0D3, Package_TO_SOT_SMD:TO-252-2, symbol Transistor_FET:QM6015D
- added Q18, Q19, Q32, Q33, Q34, Q35: AO3400, Package_TO_SOT_SMD:SOT-23_Handsoldering, symbol Transistor_FET:2N7002
- added Q4, Q5, Q6, Q9: AO3401A, Package_TO_SOT_SMD:SOT-23_Handsoldering, symbol Transistor_FET:AO3401A
- added R61, R65: 1k, Resistor_SMD:R_0805_2012Metric_Pad1.20x1.40mm_HandSolder, symbol Device:R
- added R62, R63, R64: 2K2, Resistor_SMD:R_0805_2012Metric_Pad1.20x1.40mm_HandSolder, symbol Device:R
- added U8: AMS1117-3.3, Package_TO_SOT_SMD:SOT-223-3_TabPin2, symbol Regulator_Linear:AMS1117-3.3
- C23, C24, C25, C26, C33, C34, C38, C51, C52, C53, C54, C55: footprint (none) -> Capacitor_SMD:C_0805_2012Metric_Pad1.18x1.45mm_HandSolder
- D1: footprint (none) -> LED_SMD:LED_0805_2012Metric_Pad1.15x1.40mm_HandSolder
- K2: footprint customLib:RELAY8-TH_NON-LATCH_1-COIL -> Custom:IM06D
- R100, R101, R103, R104, R105, R106, R107, R108, R109, R110, R111, R36, R37, R40, R41, R42, R47, R48, R53, R54, R55, R56, R57, R58, R59, R60, R79, R88, R89, R90, R91, R92, R93, R94, R95, R96, R97, R98, R99: footprint (none) -> Resistor_SMD:R_0805_2012Metric_Pad1.20x1.40mm_HandSolder
- U10, U11, U18, U9: footprint (none) -> Package_SO:SOIC-8-1EP_3.9x4.9mm_P1.27mm_EP2.41x3.3mm
- U6, U7: footprint (none) -> Custom:STM32F405Weact
Connections:
- net +12V: now also J13.16, Q1.3 (D), Q10.2 (D), Q4.3 (D), Q5.3 (D), Q6.3 (D), Q7.3 (D), Q9.3 (D), R61.1
- net +3.3V: now also C28.1, J13.5, R62.1, R63.1, R64.1, U8.2 (VO); no longer U6.32 (3V3), U6.34 (3V3), U6.36 (3V3)
- net +5V: now also U7.4 (5V), C27.1, J13.1, U8.3 (VI)
- net BATT: now also J13.25
- net CAN_H: now also J13.2; no longer R59.2, R60.2, U3.6 (CANL), U4.6 (CANL)
- net Curr_Filter: now also Q18.1 (G), Q19.1 (G), Q32.1 (G)
- net Drive_Supply: now also Q10.3 (S)
- net Error: now also Q1.2 (S), Q4.2 (S), Q5.2 (S), Q6.2 (S), Q7.2 (S), Q9.2 (S)
- net GND: now also U7.1 (GND), U7.2 (GND), U7.30 (GND), U7.31 (GND), U7.35 (GND), U7.59 (GND), C27.2, C28.2, D3.1 (K), J13.11, J13.13, J13.3, J13.7, Q18.2 (S), Q19.2 (S), Q32.2 (S), Q33.2 (S), Q34.2 (S), Q35.2 (S), R65.2, U8.1 (GND)
- net HallA: now also J13.8, R64.2
- net HallB: now also J13.9, R63.2
- net HallC: now also J13.10, R62.2
- net MISO_ADC_EXT2: now also J13.19
- net RX_SDA_NSS: now also J13.21
- net Ready: now also J13.15, R65.1
- net Reset: now also J13.14
- net SCK_ADC_EXT: now also J13.20
- net TX_SCI_MOSI: now also J13.18
- net Throttle_IN: now also J13.6
- net Volt_Filter: now also Q33.1 (G), Q34.1 (G), Q35.1 (G)
- net at R53.2: now also Q9.1 (G)
- net at C45.1: now also Q32.3 (D)
- net at R37.2: now also Q4.1 (G)
- net at R40.2: now also Q5.1 (G)
- net at R42.2: now also Q7.1 (G)
- net at R41.2: now also Q6.1 (G)
- net at C47.2: now also Q34.3 (D)
- net at C48.2: now also Q33.3 (D)
- net at C46.2: now also Q35.3 (D)
- net at C42.1: now also Q18.3 (D)
- net at C44.1: now also Q19.3 (D)
- net at R36.2: now also Q1.1 (G)
- net at R56.2: now also Q10.1 (G)
- net PC10_UART_RX: no longer names the net of U6.20 (C11)
- net PC10_UART_TX: no longer names the net of U6.19 (C10)
- net PC12: no longer names the net of U6.21 (C12)
- net Temp_Motor renamed TempMtr
- net TempMtr: now also J13.12
- new net: D3.2 (A), R61.2
- new net CAN_L: J13.4, R59.2, R60.2, U3.6 (CANL), U4.6 (CANL)
- new net Prech: J13.26
- no-connect marks 11 -> 27
Other:
- moved on the sheet: C23, C24, C25, C26, C33, C34, C36, C37, C38, C39, C40, C41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

Commit message: 13Nov
Parts:
- C50: footprint (none) -> Capacitor_SMD:CP_Elec_6.3x5.2
- J1, J2, J3, J4, J5, J6: footprint (none) -> Connector_PinSocket_2.54mm:PinSocket_1x03_P2.54mm_Vertical_SMD_Pin1Left
- J7, J8, J9: footprint (none) -> Connector_PinSocket_2.54mm:PinSocket_1x04_P2.54mm_Vertical_SMD_Pin1Left
- L2: value L3100u -> 100u; footprint (none) -> DR125-3R3-R:INDM1250X1250X600
Changed lines of the file:
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@@
 			)
 		)
-		(property "Footprint" ""
+		(property "Footprint" "Connector_PinSocket_2.54mm:PinSocket_1x04_P2.54mm_Vertical_SMD_Pin1Left"
 			(at 233.68 123.19 0)
 			(effects
@@
 			)
 		)
-		(property "Value" "L3100u"
+		(property "Value" "100u"
 			(at 154.94 207.772 90)
 			(effects
@@
 			)
 		)
-		(property "Footprint" ""
+		(property "Footprint" "DR125-3R3-R:INDM1250X1250X600"
 			(at 154.94 209.55 0)
 			(effects
@@
 			)
 		)
-		(property "Footprint" ""
+		(property "Footprint" "Connector_PinSocket_2.54mm:PinSocket_1x03_P2.54mm_Vertical_SMD_Pin1Left"
 			(at 219.71 118.11 0)
 			(effects
@@
 			)
 		)
-		(property "Footprint" ""
+		(property "Footprint" "Connector_PinSocket_2.54mm:PinSocket_1x04_P2.54mm_Vertical_SMD_Pin1Left"
 			(at 233.68 147.32 0)
 			(effects
@@
 			)
 		)
-		(property "Footprint" ""
+		(property "Footprint" "Connector_PinSocket_2.54mm:PinSocket_1x03_P2.54mm_Vertical_SMD_Pin1Left"
 			(at 219.71 148.59 0)
 			(effects
@@
 			)
 		)
-		(property "Footprint" ""
+		(property "Footprint" "Connector_PinSocket_2.54mm:PinSocket_1x03_P2.54mm_Vertical_SMD_Pin1Left"
 			(at 219.71 160.02 0)
 			(effects
@@
 			)
 		)
-		(property "Footprint" ""
+		(property "Footprint" "Capacitor_SMD:CP_Elec_6.3x5.2"
 			(at 113.9952 231.14 0)
 			(effects
@@
 			)
 		)
-		(property "Footprint" ""
+		(property "Footprint" "Connector_PinSocket_2.54mm:PinSocket_1x03_P2.54mm_Vertical_SMD_Pin1Left"
 			(at 219.71 168.91 0)
 			(effects
@@
 			)
 		)
-		(property "Footprint" ""
+		(property "Footprint" "Connector_PinSocket_2.54mm:PinSocket_1x03_P2.54mm_Vertical_SMD_Pin1Left"
 			(at 219.71 139.7 0)
 			(effects
@@
 			)
 		)
-		(property "Footprint" ""
+		(property "Footprint" "Connector_PinSocket_2.54mm:PinSocket_1x03_P2.54mm_Vertical_SMD_Pin1Left"
 			(at 219.71 127 0)
 			(effects
@@
 			)
 		)
-		(property "Footprint" ""
+		(property "Footprint" "Connector_PinSocket_2.54mm:PinSocket_1x04_P2.54mm_Vertical_SMD_Pin1Left"
 			(at 233.68 165.1 0)
 			(effects

Commit message: 18November
Parts:
- removed R106: 1k8, Resistor_SMD:R_0805_2012Metric_Pad1.20x1.40mm_HandSolder, symbol Device:R
- removed R108: 3k3, Resistor_SMD:R_0805_2012Metric_Pad1.20x1.40mm_HandSolder, symbol Device:R
- removed R110, R111: ref, Resistor_SMD:R_0805_2012Metric_Pad1.20x1.40mm_HandSolder, symbol Device:R
- removed U11: ~, Package_SO:SOIC-8-1EP_3.9x4.9mm_P1.27mm_EP2.41x3.3mm, symbol custom:TLV3502
- added U12: TL072H, Package_SO:SOIC-8_3.9x4.9mm_P1.27mm, symbol Device:Opamp_Dual
- C55: footprint Capacitor_SMD:C_0805_2012Metric_Pad1.18x1.45mm_HandSolder -> Capacitor_SMD:CP_Elec_5x5.4
- R107: value 2k2 -> 1k8
- R109: value 2k -> 3k3
Connections:
- net 72REG is gone; now on net Prech: C50.1, R47.1, U13.3 (VIN), U13.4 (EN/UVLO)
- net +12V: now also U12.8 (V+)
- net +5V: now also R107.1; no longer R107.2
- net ErrorVBUS: now also U12.1
- net GND: now also U12.4 (V-)
- net at R109.1: now also R107.2, U12.2 (-); no longer R107.1
- net VoltSense renamed AN_IN
- net AN_IN: now also U12.3 (+)
- no-connect marks 27 -> 69
