File: KontollerTKDNTinggi/KontollerTKDNTinggi.kicad_sch (KiCad schematic)
At the start: 130 parts, among them J1 AH_Conn, J13 6473711-1, J2 AL_Conn, J3 BH_Conn, J4 BL_Conn, J5 CH_Conn, J6 CL_Conn, J7 SignalA, J8 SignalB, J9 SignalC, K2 IM06, Q1 AO3401A, Q10 HY19P0D3, Q11 AO3401A, Q18 AO3400, Q19 AO3400, Q32 AO3400, Q33 AO3400, Q34 AO3400, Q35 AO3400, Q36 AO3400, Q4 AO3401A, Q5 AO3401A, Q6 AO3401A, Q7 AO3401A, Q9 AO3401A, U12 TL072H, U13 LM5161PWP, U14 LM2596S-5, U15 INA241A2xD, U16 INA241A2xD, U17 INA241A2xD, U3 TJA1051T-3, U4 TJA1051T-3

Commit message: 10nov
Parts:
- removed R68: 1k, Resistor_SMD:R_0805_2012Metric_Pad1.20x1.40mm_HandSolder, symbol Device:R
- R67: value 51 -> 100
Connections:
- net +3.3V: now also C33.2, C34.2, C38.2, U15.3 (REF2), U15.6 (V+), U16.3 (REF2), U16.6 (V+), U17.3 (REF2), U17.6 (V+)
- net +5V: no longer C33.2, C34.2, C38.2, U15.3 (REF2), U15.6 (V+), U16.3 (REF2), U16.6 (V+), U17.3 (REF2), U17.6 (V+)
- net Error: now also Q11.3 (D), Q36.1 (G), R55.2, U11.6 (OutB)
- net R1: now also D20.1 (K), R55.1
- net at Q36.3 (D): now also Q10.1 (G), R67.2

Commit message: test
Other:
- note added: "pppppp"
Changed lines of the file:
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@@
+		)
+	)
+	(text "pppppp\n"
+		(exclude_from_sim no)
+		(at 153.162 325.374 0)
+		(effects
+			(font
+				(size 1.27 1.27)
+			)
 		)
 	)
