File: KontollerTKDNTinggi/KontollerTKDNTinggi.kicad_pcb (KiCad board)
At the start: 4 copper layers, 277 x 148.2 mm, 139 parts, among them J1 Data_Conn, J10 GateBL, J11 A_powerSignal, J12 GateCH, J13 GateCL, J14 A_powerSignal, J16 External Switch, J2 GateAH, J3 GateAL, J4 A_powerSignal, J5 Gnd_supply, J6 V+_supply, J9 GateBH, K1 Relay_SPST-NO, Q2 AO3404, Q20 HY5110W, Q21 HY5110W, Q22 HY5110W, Q23 HY5110W, Q24 HY5110W, Q25 HY5110W, Q26 HY5110W, Q27 HY5110W, Q28 HY5110W, Q29 HY5110W, Q3 IRF9540N, Q30 HY5110W, Q31 HY5110W, Q38 HY5110W, Q39 HY5110W, Q40 HY5110W, Q41 HY5110W, Q42 HY5110W, Q43 HY5110W, Q44 HY5110W, U1 TL072, U2 AMS1117-3.3, U3 XL7015, U4 LM2596S-5

Commit message: 18November
Parts:
- removed D15: 1N5822, Diode_SMD:D_SMA_Handsoldering
- removed D16: 24V, Diode_THT:D_A-405_P10.16mm_Horizontal
- removed D17: 5V LED, LED_SMD:LED_0805_2012Metric_Pad1.15x1.40mm_HandSolder
- removed D9: 10V, Resistor_THT:R_Axial_DIN0204_L3.6mm_D1.6mm_P5.08mm_Horizontal
- removed J10: GateBL, Connector_PinSocket_2.54mm:PinSocket_1x03_P2.54mm_Vertical_SMD_Pin1Left
- removed J11, J14: A_powerSignal, Connector_PinSocket_2.54mm:PinSocket_1x04_P2.54mm_Vertical_SMD_Pin1Right
- removed J12: GateCH, Connector_PinSocket_2.54mm:PinSocket_1x03_P2.54mm_Vertical_SMD_Pin1Left
- removed J16: External Switch, Connector_Molex:Molex_Micro-Fit_3.0_43650-0200_1x02_P3.00mm_Horizontal
- removed L4: 33u, Inductor_SMD:L_10.4x10.4_H4.8
- removed Q44: HY5110W, Package_TO_SOT_THT:TO-247-3_Horizontal_TabDown
- removed TP1: +12V, TestPoint:TestPoint_Pad_2.0x2.0mm
- removed TP2: +5V, TestPoint:TestPoint_Pad_2.0x2.0mm
- added C23: 2.2u, Capacitor_SMD:C_0805_2012Metric_Pad1.18x1.45mm_HandSolder, F.Cu at (208.2, 344.1)
- added C24: 2.2u, Capacitor_SMD:C_0805_2012Metric_Pad1.18x1.45mm_HandSolder, F.Cu at (208.2, 347.1)
- added C25: 2.2u, Capacitor_SMD:C_0805_2012Metric_Pad1.18x1.45mm_HandSolder, F.Cu at (208.2, 350.1)
- added C26: 2.2u, Capacitor_SMD:C_0805_2012Metric_Pad1.18x1.45mm_HandSolder, F.Cu at (208.2, 353.1)
- added C27: 100nF, Capacitor_SMD:C_0805_2012Metric_Pad1.18x1.45mm_HandSolder, F.Cu at (208.2, 356.1)
- added C28: 47uF, Capacitor_SMD:CP_Elec_6.3x7.7, F.Cu at (243.4, 361.4)
- added C44: 15n, Capacitor_SMD:C_0805_2012Metric_Pad1.18x1.45mm_HandSolder, F.Cu at (217.8, 344.1)
- added C45: 15n, Capacitor_SMD:C_0805_2012Metric_Pad1.18x1.45mm_HandSolder, F.Cu at (217.8, 347.1)
- added C46: 100n, Capacitor_SMD:C_0805_2012Metric_Pad1.18x1.45mm_HandSolder, F.Cu at (217.8, 350.1)
- added C47: 100n, Capacitor_SMD:C_0805_2012Metric_Pad1.18x1.45mm_HandSolder, F.Cu at (217.8, 353.1)
- added C48: 100n, Capacitor_SMD:C_0805_2012Metric_Pad1.18x1.45mm_HandSolder, F.Cu at (217.8, 356.1)
- added C50: 4.7u_100V, Capacitor_SMD:CP_Elec_6.3x5.2, F.Cu at (285.7, 84.0)
- added C51: 10n, Capacitor_SMD:C_0805_2012Metric_Pad1.18x1.45mm_HandSolder, F.Cu at (281.5, 91.0)
- added C52: 2.2u, Capacitor_SMD:C_0805_2012Metric_Pad1.18x1.45mm_HandSolder, F.Cu at (283.5, 98.8)
- added C53: 100n, Capacitor_SMD:C_0805_2012Metric_Pad1.18x1.45mm_HandSolder, F.Cu at (287.5, 98.8)
- added C54: 2.2u, Capacitor_SMD:C_0805_2012Metric_Pad1.18x1.45mm_HandSolder, F.Cu at (273.0, 105.3)
- added C55: 22u_16V, Capacitor_SMD:CP_Elec_5x5.4, F.Cu at (277.8, 105.0)
- added D19: 5V LED, LED_SMD:LED_0805_2012Metric_Pad1.15x1.40mm_HandSolder, F.Cu at (258.4, 318.6)
- added D3: LED, LED_SMD:LED_0805_2012Metric_Pad1.15x1.40mm_HandSolder, F.Cu at (258.4, 315.6)
- added J7: SignalA, Connector_PinSocket_2.54mm:PinSocket_1x04_P2.54mm_Vertical_SMD_Pin1Left, F.Cu at (165.9, 358.7)
- added J8: SignalB, Connector_PinSocket_2.54mm:PinSocket_1x04_P2.54mm_Vertical_SMD_Pin1Left, F.Cu at (173.2, 358.7)
- added K2: IM06, Custom:IM06D, F.Cu at (252.0, 303.9)
- added L2: 100u, DR125-3R3-R:INDM1250X1250X600, F.Cu at (287.5, 108.0)
- added Q1: AO3401A, Package_TO_SOT_SMD:SOT-23, F.Cu at (259.8, 302.4)
- added Q10: HY19P0D3, Package_TO_SOT_SMD:TO-252-2, F.Cu at (252.6, 295.9)
- added Q18: AO3400, Package_TO_SOT_SMD:SOT-23_Handsoldering, F.Cu at (236.0, 301.4)
- added Q19: AO3400, Package_TO_SOT_SMD:SOT-23_Handsoldering, F.Cu at (242.5, 282.3)
- added Q32: AO3400, Package_TO_SOT_SMD:SOT-23_Handsoldering, F.Cu at (242.5, 287.1)
- added Q33: AO3400, Package_TO_SOT_SMD:SOT-23_Handsoldering, F.Cu at (242.5, 291.9)
- added Q34: AO3400, Package_TO_SOT_SMD:SOT-23_Handsoldering, F.Cu at (242.5, 296.6)
- added Q35: AO3400, Package_TO_SOT_SMD:SOT-23_Handsoldering, F.Cu at (242.5, 301.4)
- added Q4: AO3401A, Package_TO_SOT_SMD:SOT-23_Handsoldering, F.Cu at (236.0, 282.3)
- added Q5: AO3401A, Package_TO_SOT_SMD:SOT-23_Handsoldering, F.Cu at (236.0, 287.1)
- added Q6: AO3401A, Package_TO_SOT_SMD:SOT-23_Handsoldering, F.Cu at (236.0, 291.9)
- added Q7: AO3401A, Package_TO_SOT_SMD:SOT-23, F.Cu at (259.8, 307.0)
- added Q8: AO3404, Package_TO_SOT_SMD:SOT-23_Handsoldering, B.Cu at (327.0, 79.5)
- added Q9: AO3401A, Package_TO_SOT_SMD:SOT-23_Handsoldering, F.Cu at (236.0, 296.6)
- added R100: ref, Resistor_SMD:R_0805_2012Metric_Pad1.20x1.40mm_HandSolder, F.Cu at (248.9, 333.1)
- added R101: ref, Resistor_SMD:R_0805_2012Metric_Pad1.20x1.40mm_HandSolder, F.Cu at (248.9, 336.1)
- added R103: ref, Resistor_SMD:R_0805_2012Metric_Pad1.20x1.40mm_HandSolder, F.Cu at (253.6, 312.5)
- added R104: ref, Resistor_SMD:R_0805_2012Metric_Pad1.20x1.40mm_HandSolder, F.Cu at (253.6, 315.4)
- added R105: ref, Resistor_SMD:R_0805_2012Metric_Pad1.20x1.40mm_HandSolder, F.Cu at (253.6, 318.4)
- added R107: 1k8, Resistor_SMD:R_0805_2012Metric_Pad1.20x1.40mm_HandSolder, B.Cu at (311.0, 83.0)
- added R109: 3k3, Resistor_SMD:R_0805_2012Metric_Pad1.20x1.40mm_HandSolder, B.Cu at (310.0, 79.3)
- added R12: 56k, Resistor_SMD:R_0805_2012Metric_Pad1.20x1.40mm_HandSolder, B.Cu at (295.4, 60.5)
- added R53: 51, Resistor_SMD:R_0805_2012Metric_Pad1.20x1.40mm_HandSolder, F.Cu at (234.6, 312.5)
- added R54: 1k, Resistor_SMD:R_0805_2012Metric_Pad1.20x1.40mm_HandSolder, F.Cu at (234.6, 315.4)
- added R55: 1k, Resistor_SMD:R_0805_2012Metric_Pad1.20x1.40mm_HandSolder, F.Cu at (234.6, 318.4)
- added R56: 51, Resistor_SMD:R_0805_2012Metric_Pad1.20x1.40mm_HandSolder, F.Cu at (234.6, 321.3)
- added R57: 51, Resistor_SMD:R_0805_2012Metric_Pad1.20x1.40mm_HandSolder, F.Cu at (234.6, 324.3)
- added R58: 120, Resistor_SMD:R_0805_2012Metric_Pad1.20x1.40mm_HandSolder, F.Cu at (234.6, 327.2)
- added R59: 120, Resistor_SMD:R_0805_2012Metric_Pad1.20x1.40mm_HandSolder, F.Cu at (234.6, 330.2)
- added R60: 120, Resistor_SMD:R_0805_2012Metric_Pad1.20x1.40mm_HandSolder, F.Cu at (234.6, 333.1)
- added R61: 1k, Resistor_SMD:R_0805_2012Metric_Pad1.20x1.40mm_HandSolder, F.Cu at (234.6, 336.1)
- added R62: 2K2, Resistor_SMD:R_0805_2012Metric_Pad1.20x1.40mm_HandSolder, F.Cu at (239.4, 312.5)
- added R63: 2K2, Resistor_SMD:R_0805_2012Metric_Pad1.20x1.40mm_HandSolder, F.Cu at (239.4, 315.4)
- added R64: 2K2, Resistor_SMD:R_0805_2012Metric_Pad1.20x1.40mm_HandSolder, F.Cu at (239.4, 318.4)
- added R65: 1k, Resistor_SMD:R_0805_2012Metric_Pad1.20x1.40mm_HandSolder, F.Cu at (239.4, 321.3)
- added R79: 2k, Resistor_SMD:R_0805_2012Metric_Pad1.20x1.40mm_HandSolder, F.Cu at (278.5, 94.5)
- added R80: 1k, Resistor_SMD:R_0805_2012Metric_Pad1.20x1.40mm_HandSolder, F.Cu at (239.4, 327.2)
- added R81: 1k, Resistor_SMD:R_0805_2012Metric_Pad1.20x1.40mm_HandSolder, F.Cu at (239.4, 330.2)
- added R82: 1k, Resistor_SMD:R_0805_2012Metric_Pad1.20x1.40mm_HandSolder, F.Cu at (239.4, 333.1)
- added R83: 1k, Resistor_SMD:R_0805_2012Metric_Pad1.20x1.40mm_HandSolder, F.Cu at (239.4, 336.1)
- added R84: 1k, Resistor_SMD:R_0805_2012Metric_Pad1.20x1.40mm_HandSolder, F.Cu at (244.1, 312.5)
- added R85: 1k, Resistor_SMD:R_0805_2012Metric_Pad1.20x1.40mm_HandSolder, F.Cu at (244.1, 315.4)
- added R86: 1k, Resistor_SMD:R_0805_2012Metric_Pad1.20x1.40mm_HandSolder, F.Cu at (244.1, 318.4)
- added R87: 1k, Resistor_SMD:R_0805_2012Metric_Pad1.20x1.40mm_HandSolder, F.Cu at (244.1, 321.3)
- added R88: 1k1, Resistor_SMD:R_0805_2012Metric_Pad1.20x1.40mm_HandSolder, F.Cu at (244.1, 324.3)
- added R89: 270, Resistor_SMD:R_0805_2012Metric_Pad1.20x1.40mm_HandSolder, F.Cu at (244.1, 327.2)
- added R90: 270, Resistor_SMD:R_0805_2012Metric_Pad1.20x1.40mm_HandSolder, F.Cu at (244.1, 330.2)
- added R91: 1k1, Resistor_SMD:R_0805_2012Metric_Pad1.20x1.40mm_HandSolder, F.Cu at (244.1, 333.1)
- added R92: 270, Resistor_SMD:R_0805_2012Metric_Pad1.20x1.40mm_HandSolder, F.Cu at (244.1, 336.1)
- added R93: 1k1, Resistor_SMD:R_0805_2012Metric_Pad1.20x1.40mm_HandSolder, F.Cu at (248.9, 312.5)
- added R94: 270, Resistor_SMD:R_0805_2012Metric_Pad1.20x1.40mm_HandSolder, F.Cu at (248.9, 315.4)
- added R95: 1k1, Resistor_SMD:R_0805_2012Metric_Pad1.20x1.40mm_HandSolder, F.Cu at (248.9, 318.4)
- added R96: 270, Resistor_SMD:R_0805_2012Metric_Pad1.20x1.40mm_HandSolder, F.Cu at (248.9, 321.3)
- added R97: 270, Resistor_SMD:R_0805_2012Metric_Pad1.20x1.40mm_HandSolder, F.Cu at (248.9, 324.3)
- added R98: 1k1, Resistor_SMD:R_0805_2012Metric_Pad1.20x1.40mm_HandSolder, F.Cu at (248.9, 327.2)
- added R99: 270, Resistor_SMD:R_0805_2012Metric_Pad1.20x1.40mm_HandSolder, F.Cu at (248.9, 330.2)
- added U10: ~, Package_SO:SOIC-8-1EP_3.9x4.9mm_P1.27mm_EP2.41x3.3mm, F.Cu at (240.2, 340.9)
- added U12: TL072H, Package_SO:SOIC-8_3.9x4.9mm_P1.27mm, B.Cu at (316.7, 78.3)
- added U13: LM5161PWP, Package_SO:HTSSOP-14-1EP_4.4x5mm_P0.65mm_EP3.4x5mm_Mask3x3.1mm, F.Cu at (286.0, 92.6)
- added U14: LM2596S-5, Package_TO_SOT_SMD:TO-263-5_TabPin3, F.Cu at (314.0, 116.6)
- added U15: INA241A2xD, Package_SO:SOIC-8_3.9x4.9mm_P1.27mm, F.Cu at (276.4, 338.2)
- added U16: INA241A2xD, Package_SO:SOIC-8_3.9x4.9mm_P1.27mm, F.Cu at (248.6, 340.9)
- added U17: INA241A2xD, Package_SO:SOIC-8_3.9x4.9mm_P1.27mm, F.Cu at (248.6, 347.5)
- added U18: ~, Package_SO:SOIC-8-1EP_3.9x4.9mm_P1.27mm_EP2.41x3.3mm, F.Cu at (248.6, 354.1)
- added U5: ACS758xCB-150U-PFF, Sensor_Current:Allegro_CB_PFF, F.Cu at (274.0, 61.4)
- added U6: ~, Custom:STM32F405Weact, F.Cu at (313.1, 176.1)
- added U7: ~, Custom:STM32F405Weact, F.Cu at (313.1, 107.5)
- added U8: AMS1117-3.3, Package_TO_SOT_SMD:SOT-223-3_TabPin2, F.Cu at (257.8, 349.9)
- added U9: ~, Package_SO:SOIC-8-1EP_3.9x4.9mm_P1.27mm_EP2.41x3.3mm, F.Cu at (231.7, 354.1)
- C33: value 680uF -> 2.2u; footprint Capacitor_SMD:CP_Elec_10x10 -> Capacitor_SMD:C_0805_2012Metric_Pad1.18x1.45mm_HandSolder
- C34: value 220u -> 2.2u; footprint Capacitor_SMD:C_Elec_6.3x5.4 -> Capacitor_SMD:C_0805_2012Metric_Pad1.18x1.45mm_HandSolder
- C36: value 33u -> 680uF
- C37: value 33nF -> 220u; footprint Capacitor_SMD:C_0805_2012Metric_Pad1.18x1.45mm_HandSolder -> Capacitor_SMD:C_Elec_6.3x5.4
- C38: value 100uF -> 2.2u; footprint Capacitor_SMD:CP_Elec_8x10 -> Capacitor_SMD:C_0805_2012Metric_Pad1.18x1.45mm_HandSolder
- C39: value 1uF -> 1n
- C40: value 100nF -> 1n
- C41: value 10uF -> 1n
- C42: value 10uF -> 15n
- D1: value SS210 -> LED RED; footprint Diode_SMD:D_SMA -> LED_SMD:LED_0805_2012Metric_Pad1.15x1.40mm_HandSolder
- D14, Q2, R35: moved to B.Cu
- D18: value 12V LED -> 1N5822; footprint LED_SMD:LED_0805_2012Metric_Pad1.15x1.40mm_HandSolder -> Diode_SMD:D_SMA_Handsoldering
- J1: value Data_Conn -> AH_Conn; footprint Connector_PinSocket_2.54mm:PinSocket_2x10_P2.54mm_Vertical_SMD -> Connector_PinSocket_2.54mm:PinSocket_1x03_P2.54mm_Vertical_SMD_Pin1Left
- J13: value GateCL -> 6473711-1; footprint Connector_PinSocket_2.54mm:PinSocket_1x03_P2.54mm_Vertical_SMD_Pin1Left -> 6473711-1:TE_6473711-1
- J2: value GateAH -> AL_Conn
- J3: value GateAL -> BH_Conn
- J4: value A_powerSignal -> BL_Conn; footprint Connector_PinSocket_2.54mm:PinSocket_1x04_P2.54mm_Vertical_SMD_Pin1Right -> Connector_PinSocket_2.54mm:PinSocket_1x03_P2.54mm_Vertical_SMD_Pin1Left
- J5: value Gnd_supply -> CH_Conn; footprint Connector_PinSocket_2.54mm:PinSocket_2x02_P2.54mm_Vertical_SMD -> Connector_PinSocket_2.54mm:PinSocket_1x03_P2.54mm_Vertical_SMD_Pin1Left
- J6: value V+_supply -> CL_Conn; footprint Connector_PinSocket_2.54mm:PinSocket_2x02_P2.54mm_Vertical_SMD -> Connector_PinSocket_2.54mm:PinSocket_1x03_P2.54mm_Vertical_SMD_Pin1Left
- J9: value GateBH -> SignalB; footprint Connector_PinSocket_2.54mm:PinSocket_1x03_P2.54mm_Vertical_SMD_Pin1Left -> Connector_PinSocket_2.54mm:PinSocket_1x04_P2.54mm_Vertical_SMD_Pin1Left
- K1: footprint RELAY180LH:Untitled -> RELAY100A:RELAY100A
- L5: value 100uH -> 33u
- R36, R40: value 470K -> 51; footprint Resistor_SMD:R_1206_3216Metric_Pad1.30x1.75mm_HandSolder -> Resistor_SMD:R_0805_2012Metric_Pad1.20x1.40mm_HandSolder
- R37: value 220K -> 51; footprint Resistor_SMD:R_1206_3216Metric_Pad1.30x1.75mm_HandSolder -> Resistor_SMD:R_0805_2012Metric_Pad1.20x1.40mm_HandSolder
- R38: value 33K -> 56k; moved to B.Cu
- R39, R43: value 10K -> 2k2; moved to B.Cu
- R41: value 150K -> 51; footprint Resistor_SMD:R_1206_3216Metric_Pad1.30x1.75mm_HandSolder -> Resistor_SMD:R_0805_2012Metric_Pad1.20x1.40mm_HandSolder
- R42: value 33K -> 51; footprint Resistor_SMD:R_1206_3216Metric_Pad1.30x1.75mm_HandSolder -> Resistor_SMD:R_0805_2012Metric_Pad1.20x1.40mm_HandSolder
- R45: value 33K -> 1k; footprint Resistor_SMD:R_1206_3216Metric_Pad1.30x1.75mm_HandSolder -> Resistor_SMD:R_0805_2012Metric_Pad1.20x1.40mm_HandSolder
- R46: value 1k -> 220; footprint Resistor_SMD:R_0805_2012Metric_Pad1.20x1.40mm_HandSolder -> Resistor_SMD:R_1206_3216Metric_Pad1.30x1.75mm_HandSolder; moved to B.Cu
- R47: value 150K -> 402k; footprint Resistor_SMD:R_1206_3216Metric_Pad1.30x1.75mm_HandSolder -> Resistor_SMD:R_0805_2012Metric_Pad1.20x1.40mm_HandSolder; moved to B.Cu
- R48: value 150K -> 10k; footprint Resistor_SMD:R_1206_3216Metric_Pad1.30x1.75mm_HandSolder -> Resistor_SMD:R_0805_2012Metric_Pad1.20x1.40mm_HandSolder
- R50: value 220K -> 10K; footprint Resistor_SMD:R_1206_3216Metric_Pad1.30x1.75mm_HandSolder -> Resistor_SMD:R_0805_2012Metric_Pad1.20x1.40mm_HandSolder; moved to B.Cu
- TP3: value +3.3V -> +5V
- U1: value TL072 -> TL072H; footprint Package_SO:SO-8_3.9x4.9mm_P1.27mm -> Package_SO:SOIC-8_3.9x4.9mm_P1.27mm; moved to B.Cu
- U2: value AMS1117-3.3 -> PC817; footprint Package_TO_SOT_SMD:SOT-223-3_TabPin2 -> Package_DIP:DIP-4_W7.62mm
- U3: value XL7015 -> TJA1051T-3; footprint Package_TO_SOT_SMD:TO-252-5_TabPin6 -> Package_SO:SOIC-8_3.9x4.9mm_P1.27mm
- U4: value LM2596S-5 -> TJA1051T-3; footprint Package_TO_SOT_SMD:TO-263-5_TabPin3 -> Package_SO:SOIC-8_3.9x4.9mm_P1.27mm
- moved R34 326.9 mm to (1.88, 4.26), turned to 0 degrees
- moved J2 257.8 mm to (173.2, 347.5)
- moved J9 253.7 mm to (180.4, 358.7)
- moved J6 247.6 mm to (202.2, 347.5)
- moved J1 246.3 mm to (165.9, 347.5)
- moved C40 228.3 mm to (213.0, 353.1), turned to 0 degrees
- moved J5 216.6 mm to (194.9, 347.5)
- moved R42 215.2 mm to (229.9, 324.3), turned to 0 degrees
- moved R41 214.7 mm to (229.9, 321.3), turned to 0 degrees
- moved R40 214.4 mm to (229.9, 318.4), turned to 0 degrees
- moved C39 213.3 mm to (213.0, 350.1), turned to 0 degrees
- moved J4 212.9 mm to (187.7, 347.5)
- moved C41 210.2 mm to (213.0, 356.1), turned to 0 degrees
- moved C42 207.1 mm to (213.0, 359.1), turned to 0 degrees
- moved C38 204.8 mm to (213.0, 347.1), turned to 0 degrees
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Connections:
- net /Powerstagee/C_A renamed /Powerstagee/phaseA
- net /Powerstagee/C_B renamed /Powerstagee/phaseB
- net /Powerstagee/C_C renamed /Powerstagee/phaseC
- net Gate_BL renamed /Powerstagee/Gate_BL
- net Gate_CH renamed /Powerstagee/Gate_CH
- net VOLT_MEAS_STM32 renamed AN_IN
- C1 pad 1: V+ -> CTRL+
- C10 pad 1: V+ -> CTRL+
- C11 pad 1: V+ -> CTRL+
- C12 pad 1: V+ -> CTRL+
- C13 pad 1: V+ -> CTRL+
- C14 pad 1: V+ -> CTRL+
- C15 pad 1: V+ -> CTRL+
- C16 pad 1: V+ -> CTRL+
- C17 pad 1: V+ -> CTRL+
- C18 pad 1: V+ -> CTRL+
- C19 pad 1: V+ -> CTRL+
- C2 pad 1: V+ -> CTRL+
- C20 pad 1: V+ -> CTRL+
- C21 pad 1: V+ -> CTRL+
- C22 pad 1: V+ -> CTRL+
- C3 pad 1: V+ -> CTRL+
- C33 pad 1: +12V -> GND
- C33 pad 2: GND -> +5V
- C34 pad 1: +5V -> GND
- C34 pad 2: GND -> +5V
- C36 pad 1: V+ -> +12V
- C37 pad 1: +12V -> +5V
- C37 pad 2: Net-(U3-P$4) -> GND
- C38 pad 1: +12V -> GND
- C38 pad 2: GND -> +5V
- C39 pad 1: +12V -> GND
- C39 pad 2: GND -> /CPhaseA
- C4 pad 1: V+ -> CTRL+
- C40 pad 1: V+ -> GND
- C40 pad 2: GND -> /CPhaseB
- C41 pad 2: +5V -> /CPhaseC
- C42 pad 1: GND -> Net-(Q18-D)
- C42 pad 2: +3.3V -> /CPhaseA
- C5 pad 1: V+ -> CTRL+
- C6 pad 1: V+ -> CTRL+
- C7 pad 1: V+ -> CTRL+
- C8 pad 1: V+ -> CTRL+
- C9 pad 1: V+ -> CTRL+
- D1 pad 2: GND -> /Drive_Supply
- D14 pad 1: Net-(D14-K) -> +12V
- D18 pad 1: GND -> Net-(D18-K)
- D18 pad 2: Net-(D18-A) -> GND
- D2 pad 1: GND -> Net-(D14-A)
- H7 pad 1: BATT+ -> BATT
- J1 pad 1: /DS_A -> /Gate_AH
- J1 pad 2: /temp1 -> /Gate_AH
- J1 pad 3: /C_A -> /Gate_AH
- J13 pad 1: Gate_CL -> +5V
- J13 pad 2: Gate_CL -> /CAN_H
- J13 pad 3: Gate_CL -> GND
- J2 pad 1: Gate_AH -> /Gate_AL
- J2 pad 2: Gate_AH -> /Gate_AL
- J2 pad 3: Gate_AH -> /Gate_AL
- J3 pad 1: Gate_AL -> /Gate_BH
- J3 pad 2: Gate_AL -> /Gate_BH
- J3 pad 3: Gate_AL -> /Gate_BH
- J4 pad 1: GND -> /Gate_BL
- J4 pad 2: /PWM_AH -> /Gate_BL
- J4 pad 3: /PWM_AL -> /Gate_BL
- J5 pad 1: GND -> /Gate_CH
- J5 pad 2: GND -> /Gate_CH
- J5 pad 3: GND -> /Gate_CH
- J6 pad 1: V+ -> /Gate_CL
- J6 pad 2: V+ -> /Gate_CL
- J6 pad 3: V+ -> /Gate_CL
- J9 pad 1: Gate_BH -> /LC
- J9 pad 2: Gate_BH -> GND
- J9 pad 3: Gate_BH -> /HC
- K1 pad 14: BATT+ -> BATT
- K1 pad A1: GND -> Net-(D14-A)
- K1 pad A2: Net-(D14-K) -> +12V
- L5 pad 1: Net-(D1-K) -> Net-(D18-K)
- L5 pad 2: +12V -> +5V
- Q2 pad 1: FINISH -> Finish
- Q2 pad 2: Net-(D14-K) -> Net-(Q2-S)
- Q2 pad 3: +12V -> Net-(D14-A)
- Q20 pad 1: V+ -> CTRL+
- Q21 pad 1: V+ -> CTRL+
- Q22 pad 1: V+ -> CTRL+
- Q23 pad 1: V+ -> CTRL+
- Q24 pad 1: V+ -> CTRL+
- Q25 pad 1: V+ -> CTRL+
- Q3 pad 2: V+ -> CTRL+
- Q41 pad 1: V+ -> CTRL+
- Q42 pad 1: V+ -> CTRL+
- Q43 pad 1: V+ -> CTRL+
- R10 pad 1: Net-(J16-Pin_2) -> Prech
- R13 pad 2: Gate_AH -> /Powerstagee/Gate_AH
- R14 pad 2: Gate_AL -> /Powerstagee/Gate_AL
- R16 pad 2: Gate_AH -> /Powerstagee/Gate_AH
- R18 pad 2: Gate_AH -> /Powerstagee/Gate_AH
- R20 pad 1: Gate_AL -> /Powerstagee/Gate_AL
- R21 pad 2: Gate_BH -> /Powerstagee/Gate_BH
- R24 pad 1: Gate_CL -> /Powerstagee/Gate_CL
- R25 pad 1: Gate_BH -> /Powerstagee/Gate_BH
- R26 pad 1: Gate_BH -> /Powerstagee/Gate_BH
- R29 pad 1: Gate_AL -> /Powerstagee/Gate_AL
- R32 pad 2: Gate_CL -> /Powerstagee/Gate_CL
- R33 pad 1: Gate_CL -> /Powerstagee/Gate_CL
- R34 pad 1: Net-(D14-K) -> +12V
- R35 pad 1: FINISH -> Finish
- R36 pad 1: BATT+ -> /OvercurrentA
- R36 pad 2: Net-(R36-Pad2) -> Net-(Q1-G)
- R37 pad 1: Net-(R36-Pad2) -> /OvercurrentB
- R37 pad 2: Net-(R37-Pad2) -> Net-(Q4-G)
- R38 pad 1: Net-(R37-Pad2) -> BATT
- R38 pad 2: Net-(U1A--) -> /PreDis/Vsense
- R39 pad 1: GND -> Net-(R39-Pad1)
- R39 pad 2: Net-(U1A--) -> Net-(U1A-+)
- R40 pad 1: V+ -> /OvercurrentC
- R40 pad 2: Net-(R40-Pad2) -> Net-(Q5-G)
- R41 pad 1: Net-(R40-Pad2) -> Finish
- R41 pad 2: Net-(R41-Pad2) -> Net-(Q6-G)
- R42 pad 1: Net-(R41-Pad2) -> /Ready
- R42 pad 2: VOLT_MEAS -> Net-(Q7-G)
- R43 pad 2: VOLT_MEAS -> /PreDis/Vsense
- R45 pad 1: BATT- -> /C_A
- R45 pad 2: Net-(D9-K) -> /CPhaseA
- R46 pad 1: +5V -> Net-(R39-Pad1)
- R46 pad 2: Net-(D17-A) -> GND
- R47 pad 1: Net-(U3-P$4) -> Prech
- R47 pad 2: +12V -> Net-(U13-RON)
- R48 pad 1: GND -> +12V
- R48 pad 2: Net-(U3-P$4) -> Net-(U13-FB)
- R49 pad 1: +12V -> +5V
- R49 pad 2: Net-(D18-A) -> Net-(D19-A)
- R50 pad 1: Net-(D9-K) -> ErrorVBUS
- R50 pad 2: BATT+ -> GND
- TP3 pad 1: +3.3V -> +5V
- U1 pad 1: FINISH -> Finish
- U1 pad 2: Net-(U1A--) -> /PreDis/Vsense
- U1 pad 3: VOLT_MEAS -> Net-(U1A-+)
- U1 pad 5: VOLT_MEAS -> /PreDis/Vsense
- U2 pad 1: GND -> /Error
- U2 pad 2: +3.3V -> Net-(R54-Pad2)
- U2 pad 3: +5V -> /R2
- U3 pad 1: V+ -> /CAN_TX
- U3 pad 2: Net-(D1-K) -> GND
- U3 pad 3: GND -> +5V
- U3 pad 4: Net-(U3-P$4) -> /CAN_RX
- U3 pad 5: GND -> +3.3V
- U4 pad 1: +12V -> /CAN_TX1
- U4 pad 2: Net-(D15-K) -> GND
- U4 pad 3: GND -> +5V
- U4 pad 4: +5V -> /CAN_RX1
- U4 pad 5: GND -> +3.3V
Routing:
- net V+: track 67.0 -> 0.00 mm
- net /Powerstagee/Gate_BL: track 27.3 -> 0.00 mm
- net BATT+: track 16.9 -> 0.00 mm
- net Net-(J16-Pin_2): track 15.0 -> 0.00 mm
- added copper zone on B.Cu, net BATT
- removed copper zone on B.Cu, net BATT+
Other:
- board size 277 x 148.2 mm -> 277 x 184 mm
