File: KontollerTKDNTinggi/KontollerTKDNTinggi.kicad_pcb (KiCad board)
At the start: 4 copper layers, 277 x 148.2 mm, 139 parts, among them J1 Data_Conn, J10 GateBL, J11 A_powerSignal, J12 GateCH, J13 GateCL, J14 A_powerSignal, J16 External Switch, J2 GateAH, J3 GateAL, J4 A_powerSignal, J5 Gnd_supply, J6 V+_supply, J9 GateBH, K1 Relay_SPST-NO, Q2 AO3404, Q20 HY5110W, Q21 HY5110W, Q22 HY5110W, Q23 HY5110W, Q24 HY5110W, Q25 HY5110W, Q26 HY5110W, Q27 HY5110W, Q28 HY5110W, Q29 HY5110W, Q3 IRF9540N, Q30 HY5110W, Q31 HY5110W, Q38 HY5110W, Q39 HY5110W, Q40 HY5110W, Q41 HY5110W, Q42 HY5110W, Q43 HY5110W, Q44 HY5110W, U1 TL072, U2 AMS1117-3.3, U3 XL7015, U4 LM2596S-5

Commit message: nigeria
Parts:
- removed D15: 1N5822, Diode_SMD:D_SMA_Handsoldering
- removed D16: 24V, Diode_THT:D_A-405_P10.16mm_Horizontal
- removed D17: 5V LED, LED_SMD:LED_0805_2012Metric_Pad1.15x1.40mm_HandSolder
- removed D9: 10V, Resistor_THT:R_Axial_DIN0204_L3.6mm_D1.6mm_P5.08mm_Horizontal
- removed J10: GateBL, Connector_PinSocket_2.54mm:PinSocket_1x03_P2.54mm_Vertical_SMD_Pin1Left
- removed J11, J14: A_powerSignal, Connector_PinSocket_2.54mm:PinSocket_1x04_P2.54mm_Vertical_SMD_Pin1Right
- removed J12: GateCH, Connector_PinSocket_2.54mm:PinSocket_1x03_P2.54mm_Vertical_SMD_Pin1Left
- removed J16: External Switch, Connector_Molex:Molex_Micro-Fit_3.0_43650-0200_1x02_P3.00mm_Horizontal
- removed L4: 33u, Inductor_SMD:L_10.4x10.4_H4.8
- removed Q44: HY5110W, Package_TO_SOT_THT:TO-247-3_Horizontal_TabDown
- removed TP1: +12V, TestPoint:TestPoint_Pad_2.0x2.0mm
- removed TP2: +5V, TestPoint:TestPoint_Pad_2.0x2.0mm
- added C23: 2.2u, Capacitor_SMD:C_0805_2012Metric_Pad1.18x1.45mm_HandSolder, F.Cu at (205.2, 275.2)
- added C24: 2.2u, Capacitor_SMD:C_0805_2012Metric_Pad1.18x1.45mm_HandSolder, F.Cu at (208.2, 275.2)
- added C25: 2.2u, Capacitor_SMD:C_0805_2012Metric_Pad1.18x1.45mm_HandSolder, F.Cu at (211.2, 275.2)
- added C26: 2.2u, Capacitor_SMD:C_0805_2012Metric_Pad1.18x1.45mm_HandSolder, F.Cu at (214.2, 275.2)
- added C27: 100nF, Capacitor_SMD:C_0805_2012Metric_Pad1.18x1.45mm_HandSolder, F.Cu at (217.2, 275.2)
- added C28: 47uF, Capacitor_SMD:CP_Elec_6.3x7.7, F.Cu at (222.5, 240.1)
- added C44: 15n, Capacitor_SMD:C_0805_2012Metric_Pad1.18x1.45mm_HandSolder, F.Cu at (251.5, 180.0)
- added C45: 15n, Capacitor_SMD:C_0805_2012Metric_Pad1.18x1.45mm_HandSolder, F.Cu at (251.5, 164.0)
- added C46: 100n, Capacitor_SMD:C_0805_2012Metric_Pad1.18x1.45mm_HandSolder, F.Cu at (253.5, 188.5)
- added C47: 100n, Capacitor_SMD:C_0805_2012Metric_Pad1.18x1.45mm_HandSolder, F.Cu at (253.5, 173.0)
- added C48: 100n, Capacitor_SMD:C_0805_2012Metric_Pad1.18x1.45mm_HandSolder, F.Cu at (253.5, 157.0)
- added C50: 4.7u_100V, Capacitor_SMD:CP_Elec_6.3x5.2, F.Cu at (260.7, 83.0)
- added C51: 10n, Capacitor_SMD:C_0805_2012Metric_Pad1.18x1.45mm_HandSolder, F.Cu at (256.5, 90.0)
- added C52: 2.2u, Capacitor_SMD:C_0805_2012Metric_Pad1.18x1.45mm_HandSolder, F.Cu at (258.5, 97.8)
- added C53: 100n, Capacitor_SMD:C_0805_2012Metric_Pad1.18x1.45mm_HandSolder, F.Cu at (262.5, 97.8)
- added C54: 2.2u, Capacitor_SMD:C_0805_2012Metric_Pad1.18x1.45mm_HandSolder, F.Cu at (252.0, 110.5)
- added C55: 22u_16V, Capacitor_SMD:CP_Elec_5x5.4, F.Cu at (252.8, 104.0)
- added D19: 5V LED, LED_SMD:LED_0805_2012Metric_Pad1.15x1.40mm_HandSolder, F.Cu at (179.7, 225.0)
- added D3: LED, LED_SMD:LED_0805_2012Metric_Pad1.15x1.40mm_HandSolder, F.Cu at (176.7, 225.0)
- added J7: SignalA, Connector_PinSocket_2.54mm:PinSocket_1x04_P2.54mm_Vertical_SMD_Pin1Left, F.Cu at (66.8, 105.4)
- added J8: SignalB, Connector_PinSocket_2.54mm:PinSocket_1x04_P2.54mm_Vertical_SMD_Pin1Left, F.Cu at (126.3, 105.5)
- added K2: IM06, Custom:IM06D, F.Cu at (164.9, 231.4)
- added L2: 100u, DR125-3R3-R:INDM1250X1250X600, F.Cu at (262.5, 107.0)
- added Q1: AO3401A, Package_TO_SOT_SMD:SOT-23, F.Cu at (163.4, 223.6)
- added Q10: HY19P0D3, Package_TO_SOT_SMD:TO-252-2, F.Cu at (157.0, 230.8)
- added Q18: AO3400, Package_TO_SOT_SMD:SOT-23_Handsoldering, F.Cu at (256.5, 195.6)
- added Q19: AO3400, Package_TO_SOT_SMD:SOT-23_Handsoldering, F.Cu at (256.5, 180.1)
- added Q32: AO3400, Package_TO_SOT_SMD:SOT-23_Handsoldering, F.Cu at (256.5, 164.1)
- added Q33: AO3400, Package_TO_SOT_SMD:SOT-23_Handsoldering, F.Cu at (257.5, 157.6)
- added Q34: AO3400, Package_TO_SOT_SMD:SOT-23_Handsoldering, F.Cu at (257.5, 173.5)
- added Q35: AO3400, Package_TO_SOT_SMD:SOT-23_Handsoldering, F.Cu at (257.5, 189.1)
- added Q4: AO3401A, Package_TO_SOT_SMD:SOT-23_Handsoldering, F.Cu at (143.4, 247.4)
- added Q5: AO3401A, Package_TO_SOT_SMD:SOT-23_Handsoldering, F.Cu at (148.2, 247.4)
- added Q6: AO3401A, Package_TO_SOT_SMD:SOT-23_Handsoldering, F.Cu at (152.9, 247.4)
- added Q7: AO3401A, Package_TO_SOT_SMD:SOT-23, F.Cu at (168.1, 223.6)
- added Q8: AO3404, Package_TO_SOT_SMD:SOT-23_Handsoldering, B.Cu at (310.5, 79.5)
- added Q9: AO3401A, Package_TO_SOT_SMD:SOT-23_Handsoldering, F.Cu at (157.7, 247.4)
- added R100: ref, Resistor_SMD:R_0805_2012Metric_Pad1.20x1.40mm_HandSolder, F.Cu at (194.2, 234.6)
- added R101: ref, Resistor_SMD:R_0805_2012Metric_Pad1.20x1.40mm_HandSolder, F.Cu at (197.2, 234.6)
- added R103: ref, Resistor_SMD:R_0805_2012Metric_Pad1.20x1.40mm_HandSolder, F.Cu at (173.6, 229.8)
- added R104: ref, Resistor_SMD:R_0805_2012Metric_Pad1.20x1.40mm_HandSolder, F.Cu at (176.5, 229.8)
- added R105: ref, Resistor_SMD:R_0805_2012Metric_Pad1.20x1.40mm_HandSolder, F.Cu at (179.5, 229.8)
- added R107: 1k8, Resistor_SMD:R_0805_2012Metric_Pad1.20x1.40mm_HandSolder, B.Cu at (294.5, 83.0)
- added R109: 3k3, Resistor_SMD:R_0805_2012Metric_Pad1.20x1.40mm_HandSolder, B.Cu at (293.5, 79.3)
- added R12: 56k, Resistor_SMD:R_0805_2012Metric_Pad1.20x1.40mm_HandSolder, B.Cu at (278.9, 60.5)
- added R53: 51, Resistor_SMD:R_0805_2012Metric_Pad1.20x1.40mm_HandSolder, F.Cu at (173.6, 248.8)
- added R54: 1k, Resistor_SMD:R_0805_2012Metric_Pad1.20x1.40mm_HandSolder, F.Cu at (176.5, 248.8)
- added R55: 1k, Resistor_SMD:R_0805_2012Metric_Pad1.20x1.40mm_HandSolder, F.Cu at (179.5, 248.8)
- added R56: 51, Resistor_SMD:R_0805_2012Metric_Pad1.20x1.40mm_HandSolder, F.Cu at (182.4, 248.8)
- added R57: 51, Resistor_SMD:R_0805_2012Metric_Pad1.20x1.40mm_HandSolder, F.Cu at (185.4, 248.8)
- added R58: 120, Resistor_SMD:R_0805_2012Metric_Pad1.20x1.40mm_HandSolder, F.Cu at (188.3, 248.8)
- added R59: 120, Resistor_SMD:R_0805_2012Metric_Pad1.20x1.40mm_HandSolder, F.Cu at (191.3, 248.8)
- added R60: 120, Resistor_SMD:R_0805_2012Metric_Pad1.20x1.40mm_HandSolder, F.Cu at (194.2, 248.8)
- added R61: 1k, Resistor_SMD:R_0805_2012Metric_Pad1.20x1.40mm_HandSolder, F.Cu at (197.2, 248.8)
- added R62: 2K2, Resistor_SMD:R_0805_2012Metric_Pad1.20x1.40mm_HandSolder, F.Cu at (173.6, 244.1)
- added R63: 2K2, Resistor_SMD:R_0805_2012Metric_Pad1.20x1.40mm_HandSolder, F.Cu at (176.5, 244.1)
- added R64: 2K2, Resistor_SMD:R_0805_2012Metric_Pad1.20x1.40mm_HandSolder, F.Cu at (179.5, 244.1)
- added R65: 1k, Resistor_SMD:R_0805_2012Metric_Pad1.20x1.40mm_HandSolder, F.Cu at (182.4, 244.1)
- added R79: 2k, Resistor_SMD:R_0805_2012Metric_Pad1.20x1.40mm_HandSolder, F.Cu at (253.5, 93.5)
- added R80: 1k, Resistor_SMD:R_0805_2012Metric_Pad1.20x1.40mm_HandSolder, F.Cu at (247.0, 177.0)
- added R81: 1k, Resistor_SMD:R_0805_2012Metric_Pad1.20x1.40mm_HandSolder, F.Cu at (247.0, 161.0)
- added R82: 1k, Resistor_SMD:R_0805_2012Metric_Pad1.20x1.40mm_HandSolder, F.Cu at (247.0, 187.5)
- added R83: 1k, Resistor_SMD:R_0805_2012Metric_Pad1.20x1.40mm_HandSolder, F.Cu at (247.0, 172.0)
- added R84: 1k, Resistor_SMD:R_0805_2012Metric_Pad1.20x1.40mm_HandSolder, F.Cu at (247.0, 156.0)
- added R85: 1k, Resistor_SMD:R_0805_2012Metric_Pad1.20x1.40mm_HandSolder, F.Cu at (251.0, 188.5)
- added R86: 1k, Resistor_SMD:R_0805_2012Metric_Pad1.20x1.40mm_HandSolder, F.Cu at (251.0, 173.0)
- added R87: 1k, Resistor_SMD:R_0805_2012Metric_Pad1.20x1.40mm_HandSolder, F.Cu at (251.0, 157.0)
- added R88: 1k1, Resistor_SMD:R_0805_2012Metric_Pad1.20x1.40mm_HandSolder, F.Cu at (185.4, 239.3)
- added R89: 270, Resistor_SMD:R_0805_2012Metric_Pad1.20x1.40mm_HandSolder, F.Cu at (188.3, 239.3)
- added R90: 270, Resistor_SMD:R_0805_2012Metric_Pad1.20x1.40mm_HandSolder, F.Cu at (191.3, 239.3)
- added R91: 1k1, Resistor_SMD:R_0805_2012Metric_Pad1.20x1.40mm_HandSolder, F.Cu at (194.2, 239.3)
- added R92: 270, Resistor_SMD:R_0805_2012Metric_Pad1.20x1.40mm_HandSolder, F.Cu at (197.2, 239.3)
- added R93: 1k1, Resistor_SMD:R_0805_2012Metric_Pad1.20x1.40mm_HandSolder, F.Cu at (173.6, 234.6)
- added R94: 270, Resistor_SMD:R_0805_2012Metric_Pad1.20x1.40mm_HandSolder, F.Cu at (176.5, 234.6)
- added R95: 1k1, Resistor_SMD:R_0805_2012Metric_Pad1.20x1.40mm_HandSolder, F.Cu at (179.5, 234.6)
- added R96: 270, Resistor_SMD:R_0805_2012Metric_Pad1.20x1.40mm_HandSolder, F.Cu at (182.4, 234.6)
- added R97: 270, Resistor_SMD:R_0805_2012Metric_Pad1.20x1.40mm_HandSolder, F.Cu at (185.4, 234.6)
- added R98: 1k1, Resistor_SMD:R_0805_2012Metric_Pad1.20x1.40mm_HandSolder, F.Cu at (188.3, 234.6)
- added R99: 270, Resistor_SMD:R_0805_2012Metric_Pad1.20x1.40mm_HandSolder, F.Cu at (191.3, 234.6)
- added U10: ~, Package_SO:SOIC-8-1EP_3.9x4.9mm_P1.27mm_EP2.41x3.3mm, F.Cu at (202.0, 243.2)
- added U12: TL072H, Package_SO:SOIC-8_3.9x4.9mm_P1.27mm, B.Cu at (300.2, 78.3)
- added U13: LM5161PWP, Package_SO:HTSSOP-14-1EP_4.4x5mm_P0.65mm_EP3.4x5mm_Mask3x3.1mm, F.Cu at (261.0, 91.7)
- added U14: LM2596S-5, Package_TO_SOT_SMD:TO-263-5_TabPin3, F.Cu at (285.6, 117.2)
- added U15: INA241A2xD, Package_SO:SOIC-8_3.9x4.9mm_P1.27mm, F.Cu at (240.2, 189.4)
- added U16: INA241A2xD, Package_SO:SOIC-8_3.9x4.9mm_P1.27mm, F.Cu at (240.2, 173.9)
- added U17: INA241A2xD, Package_SO:SOIC-8_3.9x4.9mm_P1.27mm, F.Cu at (240.2, 157.9)
- added U18: ~, Package_SO:SOIC-8-1EP_3.9x4.9mm_P1.27mm_EP2.41x3.3mm, F.Cu at (215.2, 234.8)
- added U5: ACS758xCB-150U-PFF, Sensor_Current:Allegro_CB_PFF, F.Cu at (257.5, 61.4)
- added U6: ~, Custom:STM32F405Weact, F.Cu at (282.0, 171.0)
- added U7: ~, Custom:STM32F405Weact, F.Cu at (286.4, 108.6)
- added U8: AMS1117-3.3, Package_TO_SOT_SMD:SOT-223-3_TabPin2, F.Cu at (211.0, 225.6)
- added U9: ~, Package_SO:SOIC-8-1EP_3.9x4.9mm_P1.27mm_EP2.41x3.3mm, F.Cu at (215.2, 251.7)
- C33: value 680uF -> 2.2u; footprint Capacitor_SMD:CP_Elec_10x10 -> Capacitor_SMD:C_0805_2012Metric_Pad1.18x1.45mm_HandSolder
- C34: value 220u -> 2.2u; footprint Capacitor_SMD:C_Elec_6.3x5.4 -> Capacitor_SMD:C_0805_2012Metric_Pad1.18x1.45mm_HandSolder
- C36: value 33u -> 680uF
- C37: value 33nF -> 220u; footprint Capacitor_SMD:C_0805_2012Metric_Pad1.18x1.45mm_HandSolder -> Capacitor_SMD:C_Elec_6.3x5.4
- C38: value 100uF -> 2.2u; footprint Capacitor_SMD:CP_Elec_8x10 -> Capacitor_SMD:C_0805_2012Metric_Pad1.18x1.45mm_HandSolder
- C39: value 1uF -> 1n
- C40: value 100nF -> 1n
- C41: value 10uF -> 1n
- C42: value 10uF -> 15n
- D1: value SS210 -> LED RED; footprint Diode_SMD:D_SMA -> LED_SMD:LED_0805_2012Metric_Pad1.15x1.40mm_HandSolder
- D14, Q2, R35: moved to B.Cu
- D18: value 12V LED -> 1N5822; footprint LED_SMD:LED_0805_2012Metric_Pad1.15x1.40mm_HandSolder -> Diode_SMD:D_SMA_Handsoldering
- J1: value Data_Conn -> AH_Conn; footprint Connector_PinSocket_2.54mm:PinSocket_2x10_P2.54mm_Vertical_SMD -> Connector_PinSocket_2.54mm:PinSocket_1x03_P2.54mm_Vertical_SMD_Pin1Left
- J13: value GateCL -> 6473711-1; footprint Connector_PinSocket_2.54mm:PinSocket_1x03_P2.54mm_Vertical_SMD_Pin1Left -> 6473711-1:TE_6473711-1
- J2: value GateAH -> AL_Conn
- J3: value GateAL -> BH_Conn
- J4: value A_powerSignal -> BL_Conn; footprint Connector_PinSocket_2.54mm:PinSocket_1x04_P2.54mm_Vertical_SMD_Pin1Right -> Connector_PinSocket_2.54mm:PinSocket_1x03_P2.54mm_Vertical_SMD_Pin1Left
- J5: value Gnd_supply -> CH_Conn; footprint Connector_PinSocket_2.54mm:PinSocket_2x02_P2.54mm_Vertical_SMD -> Connector_PinSocket_2.54mm:PinSocket_1x03_P2.54mm_Vertical_SMD_Pin1Left
- J6: value V+_supply -> CL_Conn; footprint Connector_PinSocket_2.54mm:PinSocket_2x02_P2.54mm_Vertical_SMD -> Connector_PinSocket_2.54mm:PinSocket_1x03_P2.54mm_Vertical_SMD_Pin1Left
- J9: value GateBH -> SignalC; footprint Connector_PinSocket_2.54mm:PinSocket_1x03_P2.54mm_Vertical_SMD_Pin1Left -> Connector_PinSocket_2.54mm:PinSocket_1x04_P2.54mm_Vertical_SMD_Pin1Left
- K1: footprint RELAY180LH:Untitled -> RELAY100A:RELAY100A
- L5: value 100uH -> 33u
- R15, R17, R19: footprint Resistor_SMD:R_0805_2012Metric_Pad1.20x1.40mm_HandSolder -> Resistor_THT:R_Axial_DIN0204_L3.6mm_D1.6mm_P1.90mm_Vertical
- R36, R40: value 470K -> 51; footprint Resistor_SMD:R_1206_3216Metric_Pad1.30x1.75mm_HandSolder -> Resistor_SMD:R_0805_2012Metric_Pad1.20x1.40mm_HandSolder
- R37: value 220K -> 51; footprint Resistor_SMD:R_1206_3216Metric_Pad1.30x1.75mm_HandSolder -> Resistor_SMD:R_0805_2012Metric_Pad1.20x1.40mm_HandSolder
- R38: value 33K -> 56k; moved to B.Cu
- R39, R43: value 10K -> 2k2; moved to B.Cu
- R41: value 150K -> 51; footprint Resistor_SMD:R_1206_3216Metric_Pad1.30x1.75mm_HandSolder -> Resistor_SMD:R_0805_2012Metric_Pad1.20x1.40mm_HandSolder
- R42: value 33K -> 51; footprint Resistor_SMD:R_1206_3216Metric_Pad1.30x1.75mm_HandSolder -> Resistor_SMD:R_0805_2012Metric_Pad1.20x1.40mm_HandSolder
- R45: value 33K -> 1k; footprint Resistor_SMD:R_1206_3216Metric_Pad1.30x1.75mm_HandSolder -> Resistor_SMD:R_0805_2012Metric_Pad1.20x1.40mm_HandSolder
- R46: value 1k -> 220; footprint Resistor_SMD:R_0805_2012Metric_Pad1.20x1.40mm_HandSolder -> Resistor_SMD:R_1206_3216Metric_Pad1.30x1.75mm_HandSolder; moved to B.Cu
- R47: value 150K -> 402k; footprint Resistor_SMD:R_1206_3216Metric_Pad1.30x1.75mm_HandSolder -> Resistor_SMD:R_0805_2012Metric_Pad1.20x1.40mm_HandSolder; moved to B.Cu
- R48: value 150K -> 10k; footprint Resistor_SMD:R_1206_3216Metric_Pad1.30x1.75mm_HandSolder -> Resistor_SMD:R_0805_2012Metric_Pad1.20x1.40mm_HandSolder
- R50: value 220K -> 10K; footprint Resistor_SMD:R_1206_3216Metric_Pad1.30x1.75mm_HandSolder -> Resistor_SMD:R_0805_2012Metric_Pad1.20x1.40mm_HandSolder; moved to B.Cu
- TP3: value +3.3V -> +5V
- U1: value TL072 -> TL072H; footprint Package_SO:SO-8_3.9x4.9mm_P1.27mm -> Package_SO:SOIC-8_3.9x4.9mm_P1.27mm; moved to B.Cu
- U2: value AMS1117-3.3 -> PC817; footprint Package_TO_SOT_SMD:SOT-223-3_TabPin2 -> Package_DIP:DIP-4_W7.62mm
- U3: value XL7015 -> TJA1051T-3; footprint Package_TO_SOT_SMD:TO-252-5_TabPin6 -> Package_SO:SOIC-8_3.9x4.9mm_P1.27mm
- U4: value LM2596S-5 -> TJA1051T-3; footprint Package_TO_SOT_SMD:TO-263-5_TabPin3 -> Package_SO:SOIC-8_3.9x4.9mm_P1.27mm
- moved R34 326.9 mm to (1.88, 4.26), turned to 0 degrees
- moved J1 223.9 mm to (71.1, 79.5), turned to 180 degrees
- moved R36 192.1 mm to (173.6, 253.6), turned to 90 degrees
- moved R40 192.0 mm to (179.5, 253.6), turned to 90 degrees
- moved R41 185.7 mm to (182.4, 253.6), turned to 90 degrees
- moved R37 185.5 mm to (176.5, 253.6), turned to 90 degrees
- moved R42 179.4 mm to (185.4, 253.6), turned to 90 degrees
- moved C16 178.0 mm to (83.2, 101.3), turned to -90 degrees
- moved R49 150.0 mm to (197.2, 253.6), turned to 90 degrees
- moved U2 146.1 mm to (166.8, 249.0), turned to 90 degrees
- moved TP3 127.5 mm to (183.2, 225.4), turned to 90 degrees
- moved J5 123.3 mm to (189.0, 79.0), turned to 180 degrees
- moved J13 120.9 mm to (313.0, 159.7), turned to 90 degrees
- moved C17 119.9 mm to (143.2, 101.4), turned to -90 degrees
- moved J3 107.8 mm to (130.5, 79.5), turned to 180 degrees
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Connections:
- net /Powerstagee/C_A renamed PA
- net /Powerstagee/C_B renamed PB
- net /Powerstagee/C_C renamed PC
- net /Powerstagee/DS_A renamed DS_A
- net /Powerstagee/DS_B renamed DS_B
- net /Powerstagee/DS_C renamed DS_C
- net VOLT_MEAS_STM32 renamed AN_IN
- C1 pad 1: V+ -> CTRL+
- C10 pad 1: V+ -> CTRL+
- C11 pad 1: V+ -> CTRL+
- C12 pad 1: V+ -> CTRL+
- C13 pad 1: V+ -> CTRL+
- C14 pad 1: V+ -> CTRL+
- C15 pad 1: V+ -> CTRL+
- C16 pad 1: V+ -> CTRL+
- C17 pad 1: V+ -> CTRL+
- C18 pad 1: V+ -> CTRL+
- C19 pad 1: V+ -> CTRL+
- C2 pad 1: V+ -> CTRL+
- C20 pad 1: V+ -> CTRL+
- C21 pad 1: V+ -> CTRL+
- C22 pad 1: V+ -> CTRL+
- C3 pad 1: V+ -> CTRL+
- C33 pad 1: +12V -> GND
- C33 pad 2: GND -> +5V
- C34 pad 1: +5V -> GND
- C34 pad 2: GND -> +5V
- C36 pad 1: V+ -> +12V
- C37 pad 1: +12V -> +5V
- C37 pad 2: Net-(U3-P$4) -> GND
- C38 pad 1: +12V -> GND
- C38 pad 2: GND -> +5V
- C39 pad 1: +12V -> GND
- C39 pad 2: GND -> /CPhaseA
- C4 pad 1: V+ -> CTRL+
- C40 pad 1: V+ -> GND
- C40 pad 2: GND -> /CPhaseB
- C41 pad 2: +5V -> /CPhaseC
- C42 pad 1: GND -> Net-(Q18-D)
- C42 pad 2: +3.3V -> /CPhaseA
- C5 pad 1: V+ -> CTRL+
- C6 pad 1: V+ -> CTRL+
- C7 pad 1: V+ -> CTRL+
- C8 pad 1: V+ -> CTRL+
- C9 pad 1: V+ -> CTRL+
- D1 pad 2: GND -> /Drive_Supply
- D14 pad 1: Net-(D14-K) -> +12V
- D18 pad 1: GND -> Net-(D18-K)
- D18 pad 2: Net-(D18-A) -> GND
- D2 pad 1: GND -> Net-(D14-A)
- H7 pad 1: BATT+ -> BATT
- J1 pad 1: /DS_A -> Gate_AH
- J1 pad 2: /temp1 -> Gate_AH
- J1 pad 3: /C_A -> Gate_AH
- J13 pad 1: Gate_CL -> +5V
- J13 pad 2: Gate_CL -> /CAN_H
- J13 pad 3: Gate_CL -> GND
- J2 pad 1: Gate_AH -> Gate_AL
- J2 pad 2: Gate_AH -> Gate_AL
- J2 pad 3: Gate_AH -> Gate_AL
- J3 pad 1: Gate_AL -> Gate_BH
- J3 pad 2: Gate_AL -> Gate_BH
- J3 pad 3: Gate_AL -> Gate_BH
- J4 pad 1: GND -> Gate_BL
- J4 pad 2: /PWM_AH -> Gate_BL
- J4 pad 3: /PWM_AL -> Gate_BL
- J5 pad 1: GND -> Gate_CH
- J5 pad 2: GND -> Gate_CH
- J5 pad 3: GND -> Gate_CH
- J6 pad 1: V+ -> Gate_CL
- J6 pad 2: V+ -> Gate_CL
- J6 pad 3: V+ -> Gate_CL
- J9 pad 1: Gate_BH -> /LC
- J9 pad 2: Gate_BH -> GND
- J9 pad 3: Gate_BH -> /HC
- K1 pad 14: BATT+ -> BATT
- K1 pad A1: GND -> Net-(D14-A)
- K1 pad A2: Net-(D14-K) -> +12V
- L5 pad 1: Net-(D1-K) -> Net-(D18-K)
- L5 pad 2: +12V -> +5V
- Q2 pad 1: FINISH -> Finish
- Q2 pad 2: Net-(D14-K) -> Net-(Q2-S)
- Q2 pad 3: +12V -> Net-(D14-A)
- Q20 pad 1: V+ -> CTRL+
- Q21 pad 1: V+ -> CTRL+
- Q22 pad 1: V+ -> CTRL+
- Q23 pad 1: V+ -> CTRL+
- Q24 pad 1: V+ -> CTRL+
- Q25 pad 1: V+ -> CTRL+
- Q3 pad 2: V+ -> CTRL+
- Q41 pad 1: V+ -> CTRL+
- Q42 pad 1: V+ -> CTRL+
- Q43 pad 1: V+ -> CTRL+
- R10 pad 1: Net-(J16-Pin_2) -> Prech
- R15 pad 2: /Powerstagee/temp1 -> TempA
- R17 pad 2: /Powerstagee/temp2 -> TempB
- R19 pad 2: /Powerstagee/temp3 -> TempC
- R34 pad 1: Net-(D14-K) -> +12V
- R35 pad 1: FINISH -> Finish
- R36 pad 1: BATT+ -> /OvercurrentA
- R36 pad 2: Net-(R36-Pad2) -> Net-(Q1-G)
- R37 pad 1: Net-(R36-Pad2) -> /OvercurrentB
- R37 pad 2: Net-(R37-Pad2) -> Net-(Q4-G)
- R38 pad 1: Net-(R37-Pad2) -> BATT
- R38 pad 2: Net-(U1A--) -> /PreDis/Vsense
- R39 pad 1: GND -> Net-(R39-Pad1)
- R39 pad 2: Net-(U1A--) -> Net-(U1A-+)
- R40 pad 1: V+ -> /OvercurrentC
- R40 pad 2: Net-(R40-Pad2) -> Net-(Q5-G)
- R41 pad 1: Net-(R40-Pad2) -> Finish
- R41 pad 2: Net-(R41-Pad2) -> Net-(Q6-G)
- R42 pad 1: Net-(R41-Pad2) -> /Ready
- R42 pad 2: VOLT_MEAS -> Net-(Q7-G)
- R43 pad 2: VOLT_MEAS -> /PreDis/Vsense
- R45 pad 1: BATT- -> /C_A
- R45 pad 2: Net-(D9-K) -> /CPhaseA
- R46 pad 1: +5V -> Net-(R39-Pad1)
- R46 pad 2: Net-(D17-A) -> GND
- R47 pad 1: Net-(U3-P$4) -> Prech
- R47 pad 2: +12V -> Net-(U13-RON)
- R48 pad 1: GND -> +12V
- R48 pad 2: Net-(U3-P$4) -> Net-(U13-FB)
- R49 pad 1: +12V -> +5V
- R49 pad 2: Net-(D18-A) -> Net-(D19-A)
- R50 pad 1: Net-(D9-K) -> ErrorVBUS
- R50 pad 2: BATT+ -> GND
- TP3 pad 1: +3.3V -> +5V
- U1 pad 1: FINISH -> Finish
- U1 pad 2: Net-(U1A--) -> /PreDis/Vsense
- U1 pad 3: VOLT_MEAS -> Net-(U1A-+)
- U1 pad 5: VOLT_MEAS -> /PreDis/Vsense
- U2 pad 1: GND -> /Error
- U2 pad 2: +3.3V -> Net-(R54-Pad2)
- U2 pad 3: +5V -> /R2
- U3 pad 1: V+ -> /CAN_TX
- U3 pad 2: Net-(D1-K) -> GND
- U3 pad 3: GND -> +5V
- U3 pad 4: Net-(U3-P$4) -> /CAN_RX
- U3 pad 5: GND -> +3.3V
- U4 pad 1: +12V -> /CAN_TX1
- U4 pad 2: Net-(D15-K) -> GND
- U4 pad 3: GND -> +5V
- U4 pad 4: +5V -> /CAN_RX1
- U4 pad 5: GND -> +3.3V
Routing:
- net /HA: track 0.00 -> 92.0 mm
- net /LA: track 0.00 -> 86.3 mm
- net V+: track 67.0 -> 0.00 mm
- net Gate_AL: track 0.00 -> 55.4 mm
- net TempB: track 0.00 -> 34.3 mm
- net TempC: track 0.00 -> 28.0 mm
- net Gate_BL: track 27.3 -> 54.5 mm
- net BATT+: track 16.9 -> 0.00 mm
- net Net-(J16-Pin_2): track 15.0 -> 0.00 mm
- net Net-(Q26-G): track 0.00 -> 5.26 mm
- net /HB: track 0.00 -> 1.81 mm
- net Net-(Q43-G): track 5.37 -> 6.59 mm
- net PC: vias 0 -> 1
- net GND: vias 0 -> 75
- net DS_C: vias 0 -> 1
- added copper zone on B.Cu, net BATT
- added copper zone on B.Cu, net CTRL+
- added copper zone on B.Cu, net DS_A
- added copper zone on B.Cu, net DS_B
- added copper zone on B.Cu, net DS_C
- added copper zone on B.Cu, net PA
- added copper zone on B.Cu, net PB
- added copper zone on B.Cu, net PC
- removed copper zone on B.Cu, net /C_A
- removed copper zone on B.Cu, net /C_B
- removed copper zone on B.Cu, net /C_C
- removed copper zone on B.Cu, net /DS_A
- removed copper zone on B.Cu, net /DS_B
- removed copper zone on B.Cu, net /DS_C
- removed copper zone on B.Cu, net BATT+
- removed copper zone on B.Cu, net V+
Other:
- board size 277 x 148.2 mm -> 282 x 173.8 mm

Commit message: mendekatifix
Parts:
- removed Q3: IRF9540N, Package_TO_SOT_THT:TO-220-3_Vertical
- removed U2: PC817, Package_DIP:DIP-4_W7.62mm
- removed U8: AMS1117-3.3, Package_TO_SOT_SMD:SOT-223-3_TabPin2
- added C29: 2.2u, Capacitor_SMD:C_0805_2012Metric_Pad1.18x1.45mm_HandSolder, F.Cu at (275.0, 217.7)
- added D20: 1N5822, Diode_SMD:D_SMA_Handsoldering, F.Cu at (283.2, 127.7)
- added FDA117: ~, Custom:FDA117, F.Cu at (254.1, 77.2)
- added Q11: AO3401A, Package_TO_SOT_SMD:SOT-23_Handsoldering, F.Cu at (284.7, 135.6)
- added Q13: IXTY1R6N100D2, Package_TO_SOT_SMD:TO-252-2, F.Cu at (254.6, 68.6)
- added Q36: AO3400, Package_TO_SOT_SMD:SOT-23_Handsoldering, F.Cu at (246.8, 53.7)
- added R102: 1k1, Resistor_SMD:R_0805_2012Metric_Pad1.20x1.40mm_HandSolder, F.Cu at (259.8, 150.3)
- added R44: R, Resistor_SMD:R_0805_2012Metric_Pad1.20x1.40mm_HandSolder, F.Cu at (299.6, 132.2)
- added R66: 10k, Resistor_SMD:R_0805_2012Metric_Pad1.20x1.40mm_HandSolder, F.Cu at (279.8, 217.5)
- added R67: 51, Resistor_SMD:R_0805_2012Metric_Pad1.20x1.40mm_HandSolder, F.Cu at (236.8, 59.2)
- added R68: 1k, Resistor_SMD:R_0805_2012Metric_Pad1.20x1.40mm_HandSolder, F.Cu at (241.4, 59.2)
- added TP4: +12V, TestPoint:TestPoint_Pad_2.0x2.0mm, F.Cu at (303.2, 120.0)
- added U11: ~, Package_SO:SOIC-8_3.9x4.9mm_P1.27mm, F.Cu at (293.2, 135.2)
- C27: value 100nF -> 2.2u
- C28: value 47uF -> 2.2u; footprint Capacitor_SMD:CP_Elec_6.3x7.7 -> Capacitor_SMD:C_0805_2012Metric_Pad1.18x1.45mm_HandSolder
- Q1, Q7: footprint Package_TO_SOT_SMD:SOT-23 -> Package_TO_SOT_SMD:SOT-23_Handsoldering
- R10: value 500 -> 1k; footprint Package_TO_SOT_THT:TO-247-2_Horizontal_TabDown -> Resistor_THT:R_Axial_DIN0918_L18.0mm_D9.0mm_P30.48mm_Horizontal
- R11: footprint Resistor_SMD:R_2816_7142Metric_Pad3.20x4.45mm_HandSolder -> Resistor_THT:R_Axial_DIN0617_L17.0mm_D6.0mm_P20.32mm_Horizontal
- R15, R17, R19: value NTC 10K -> PTC
- R51: value 1K -> 10K
- R52: value 1K -> 10k
- R54, R55: value 1k -> R
- R56: value 51 -> R
- R57: value 51 -> 560
- U10, U18, U9: footprint Package_SO:SOIC-8-1EP_3.9x4.9mm_P1.27mm_EP2.41x3.3mm -> Package_SO:SOIC-8_3.9x4.9mm_P1.27mm
- moved R34 310.5 mm to (301.8, 85.0), turned to -90 degrees
- moved D1 203.2 mm to (250.6, 59.0), turned to 90 degrees
- moved R58 198.9 mm to (247.8, 59.0)
- moved Q10 198.7 mm to (238.5, 49.6)
- moved R57 188.8 mm to (263.2, 76.7)
- moved R49 187.6 mm to (281.5, 86.0), turned to -90 degrees
- moved R11 179.8 mm to (269.6, 77.4), turned to 90 degrees
- moved Q6 178.5 mm to (302.7, 150.3)
- moved TP3 174.2 mm to (281.5, 81.5)
- moved K2 174.0 mm to (306.7, 130.6), turned to -90 degrees
- moved Q5 173.5 mm to (287.2, 143.6)
- moved D3 171.5 mm to (303.2, 109.2), turned to -90 degrees
- moved R61 171.1 mm to (303.2, 114.5)
- moved D19 168.5 mm to (281.5, 90.8)
- moved C23 166.6 mm to (259.8, 117.8)
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Connections:
- C27 pad 1: +5V -> +3.3V
- C27 pad 2: GND -> TempC
- C28 pad 2: GND -> TempB
- K2 pad 5: Net-(K2-Pad5) -> /R1
- K2 pad 6: /R2 -> +12V
- K2 pad 7: /Error -> unconnected-(K2-Pad7)
- Q10 pad 2: +12V -> /Drive_Supply
- Q10 pad 3: /Drive_Supply -> +12V
- R107 pad 2: Net-(U12A--) -> Net-(U12A-+)
- R109 pad 1: Net-(U12A--) -> Net-(U12A-+)
- R11 pad 1: GND -> Net-(Q13-D)
- R11 pad 2: Net-(Q3-S) -> CTRL+
- R15 pad 1: GND -> +3.3V
- R17 pad 1: GND -> +3.3V
- R19 pad 1: GND -> +3.3V
- R51 pad 1: Net-(Q3-G) -> TempC
- R51 pad 2: +12V -> GND
- R52 pad 1: Net-(Q3-G) -> TempB
- R54 pad 1: GND -> Net-(U11-+In2)
- R54 pad 2: Net-(R54-Pad2) -> GND
- R55 pad 1: GND -> Net-(D20-K)
- R55 pad 2: /R2 -> Net-(Q11-D)
- R56 pad 1: /R2 -> +12V
- R56 pad 2: Net-(Q10-G) -> Net-(D20-A)
- R57 pad 1: Net-(K2-Pad5) -> +5V
- R57 pad 2: +12V -> Net-(FDA117-in+)
- U12 pad 2: Net-(U12A--) -> AN_IN
- U12 pad 3: AN_IN -> Net-(U12A-+)
- U6 pad 32: unconnected-(U6-3V3-Pad32) -> +3.3V
- U6 pad 34: unconnected-(U6-3V3-Pad34) -> +3.3V
- U6 pad 36: unconnected-(U6-3V3-Pad36) -> +3.3V
- U7 pad 32: unconnected-(U7-3V3-Pad32) -> +3.3V
- U7 pad 34: unconnected-(U7-3V3-Pad34) -> +3.3V
- U7 pad 36: unconnected-(U7-3V3-Pad36) -> +3.3V
Routing:
- net /HB: track 1.81 -> 245.0 mm
- net /HA: track 92.0 -> 329.5 mm, vias 0 -> 1
- net /LB: track 0.00 -> 226.2 mm
- net /LA: track 86.3 -> 309.8 mm
- net PA: track 0.00 -> 184.9 mm, vias 0 -> 1
- net DS_A: track 0.00 -> 184.3 mm, vias 0 -> 1
- net /HC: track 0.00 -> 183.9 mm
- net /LC: track 0.00 -> 173.4 mm
- net TempB: track 34.3 -> 169.5 mm
- net DS_B: track 0.00 -> 109.6 mm, vias 0 -> 1
- net PB: track 0.00 -> 109.4 mm, vias 0 -> 1
- net TempC: track 28.0 -> 72.9 mm
- net DS_C: track 0.00 -> 35.6 mm
- net PC: track 0.00 -> 35.2 mm
- net TempA: track 0.00 -> 27.0 mm, vias 0 -> 1
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- added copper zone on In2.Cu, net GND
- removed copper zone on B.Cu, net BATT
Other:
- board size 282 x 173.8 mm -> 285.6 x 172.1 mm

Commit message: 10nov
Parts:
- moved J13 0.81 mm to (317.0, 161.2)
Other:
- board size 285.6 x 172.1 mm -> 262.6 x 172.1 mm
Changed lines of the file:
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@@
 	(footprint "6473711-1:TE_6473711-1"
 		(layer "F.Cu")
-		(at 317 160.4375 90)
+		(at 317 161.25 90)
 		(property "Reference" "J13"
 			(at -26.83555 -5.14485 90)
@@
 	(gr_rect
 		(start 58.42 31.695)
-		(end 344.045 203.750879)
+		(end 321.045 203.750879)
 		(stroke
 			(width 0.05)
