File: KontollerTKDNTinggi/Powerstagee'.kicad_sch (KiCad schematic)
At the start: 71 parts, among them Q20 HY5110W, Q21 HY5110W, Q22 HY5110W, Q23 HY5110W, Q24 HY5110W, Q25 HY5110W, Q26 HY5110W, Q27 HY5110W, Q28 HY5110W, Q29 HY5110W, Q30 HY5110W, Q31 HY5110W, Q38 HY5110W, Q39 HY5110W, Q40 HY5110W, Q41 HY5110W, Q42 HY5110W, Q43 HY5110W, U5 ACS758xCB-150U-PFF

Commit message: 18November
Changed lines of the file:
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@@
+		)
+	)
+	(global_label "DC_Current"
+		(shape input)
+		(at 50.8 21.59 0)
+		(fields_autoplaced yes)
+		(effects
+			(font
+				(size 1.27 1.27)
+			)
+			(justify left)
+		)
+		(property "Intersheetrefs" "${INTERSHEET_REFS}"
+			(at 64.2475 21.59 0)
+			(effects
+				(font
+					(size 1.27 1.27)
+				)
+				(justify left)
+				(hide yes)
+			)
 		)
 	)
@@
 		)
 	)
-	(hierarchical_label "DC_Current"
-		(shape input)
-		(at 50.8 21.59 0)
-		(effects
-			(font
-				(size 1.27 1.27)
-				(thickness 0.1588)
-			)
-			(justify left)
-		)
-	)
