File: KontollerTKDNTinggi/Powerstagee'.kicad_sch (KiCad schematic)
At the start: 70 parts, among them Q20 HY5110W, Q21 HY5110W, Q22 HY5110W, Q23 HY5110W, Q24 HY5110W, Q25 HY5110W, Q26 HY5110W, Q27 HY5110W, Q28 HY5110W, Q29 HY5110W, Q30 HY5110W, Q31 HY5110W, Q38 HY5110W, Q39 HY5110W, Q40 HY5110W, Q41 HY5110W, Q42 HY5110W, Q43 HY5110W

Commit message: 11Nov
Parts:
- added U5: ACS758xCB-150U-PFF, Sensor_Current:Allegro_CB_PFF, symbol Sensor_Current:ACS758xCB-150U-PFF
Connections:
- net GND: now also U5.2 (GND)
- net V+: now also U5.4 (IP+); no longer C1.1, C10.1, C11.1, C12.1, C13.1, C14.1, C15.1, C16.1, C17.1, C18.1, C19.1, C2.1, C20.1, C21.1, C22.1, C3.1, C4.1, C5.1, C6.1, C7.1, C8.1, C9.1, Q20.1 (D), Q21.1 (D), Q22.1 (D), Q23.1 (D), Q24.1 (D), Q25.1 (D), Q41.1 (D), Q42.1 (D), Q43.1 (D)
- new net +3.3V: U5.1 (VCC)
- new net CTRL+: C1.1, C10.1, C11.1, C12.1, C13.1, C14.1, C15.1, C16.1, C17.1, C18.1, C19.1, C2.1, C20.1, C21.1, C22.1, C3.1, C4.1, C5.1, C6.1, C7.1, C8.1, C9.1, Q20.1 (D), Q21.1 (D), Q22.1 (D), Q23.1 (D), Q24.1 (D), Q25.1 (D), Q41.1 (D), Q42.1 (D), Q43.1 (D), U5.5 (IP-)
- new net DC_Current: U5.3 (VIOUT)

Commit message: nigeria
Parts:
- R15, R17, R19: footprint Resistor_SMD:R_0805_2012Metric_Pad1.20x1.40mm_HandSolder -> Resistor_THT:R_Axial_DIN0204_L3.6mm_D1.6mm_P1.90mm_Vertical
Connections:
- net phaseA renamed PA
- net phaseB renamed PB
- net phaseC renamed PC
- net temp1 renamed TempA
- net temp2 renamed TempB
- net temp3 renamed TempC

Commit message: mendekatifix
Parts:
- added C27, C28, C29: 2.2u, Capacitor_SMD:C_0805_2012Metric_Pad1.18x1.45mm_HandSolder, symbol Device:C
- added R51: 10K, Resistor_SMD:R_0805_2012Metric_Pad1.20x1.40mm_HandSolder, symbol Device:R
- added R52, R66: 10k, Resistor_SMD:R_0805_2012Metric_Pad1.20x1.40mm_HandSolder, symbol Device:R
- R15, R17, R19: value NTC 10K -> PTC
Connections:
- net +3.3V: now also R15.1, R17.1, R19.1, C27.1, C28.1, C29.1
- net GND: now also R51.2, R52.2, R66.2; no longer R15.1, R17.1, R19.1
- net TempA: now also C29.2, R66.1
- net TempB: now also C28.2, R52.1
- net TempC: now also C27.2, R51.1
Other:
- moved on the sheet: R15, R17, R19
