File: KontollerTKDNTinggi/PreDis.kicad_sch (KiCad schematic)
At the start: 21 parts, among them K1 Relay_SPST-NO, Q2 AO3404, Q3 IRF9540N, Q8 AO3404, U1 TL072H

Commit message: 11Nov
Connections:
- net +12V: now also D14.1 (K), K1.A2, R34.1; no longer Q2.3 (D)
- net GND: now also Q8.2 (S); no longer D14.2 (A), D2.1 (K), K1.A1
- net V+: no longer Q3.2 (D)
- new net: D14.2 (A), D2.1 (K), K1.A1, Q2.3 (D)
- new net CTRL+: Q3.2 (D)
Other:
- moved on the sheet: D14, D2, Q2, Q8, R34, R35, R50

Commit message: ganticonnector
Parts:
- R12: footprint (none) -> Resistor_SMD:R_0805_2012Metric_Pad1.20x1.40mm_HandSolder
- U1: footprint (none) -> Package_SO:SOIC-8-1EP_3.9x4.9mm_P1.27mm_EP2.62x3.51mm
Changed lines of the file:
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@@
 		)
 	)
-	(hierarchical_label "CTRL"
+	(hierarchical_label "Prech"
 		(shape input)
 		(at 93.98 40.64 90)
@@
 			)
 		)
-		(property "Footprint" ""
+		(property "Footprint" "Resistor_SMD:R_0805_2012Metric_Pad1.20x1.40mm_HandSolder"
 			(at 92.71 75.438 90)
 			(effects
@@
 			)
 		)
-		(property "Footprint" ""
+		(property "Footprint" "Package_SO:SOIC-8-1EP_3.9x4.9mm_P1.27mm_EP2.62x3.51mm"
 			(at 123.19 90.17 0)
 			(effects
@@
 			)
 		)
-		(property "Footprint" ""
+		(property "Footprint" "Package_SO:SOIC-8-1EP_3.9x4.9mm_P1.27mm_EP2.62x3.51mm"
 			(at 124.46 110.49 0)
 			(effects
@@
 			)
 		)
-		(property "Footprint" ""
+		(property "Footprint" "Package_SO:SOIC-8-1EP_3.9x4.9mm_P1.27mm_EP2.62x3.51mm"
 			(at 123.19 90.17 0)
 			(effects

Commit message: nigeria
Parts:
- K1: footprint RELAY180LH:Untitled -> RELAY100A:RELAY100A
- U1: footprint Package_SO:SOIC-8-1EP_3.9x4.9mm_P1.27mm_EP2.62x3.51mm -> Package_SO:SOIC-8_3.9x4.9mm_P1.27mm
Connections:
- net 72REG renamed Prech
- net VoltSense renamed AN_IN
Changed lines of the file:
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@@
-	)
-	(junction
-		(at 87.63 45.72)
-		(diameter 0)
-		(color 0 0 0 0)
 	)
 	(junction
@@
 		(color 0 0 0 0)
 	)
-	(junction
-		(at 96.52 45.72)
-		(diameter 0)
-		(color 0 0 0 0)
-	)
 	(wire
 		(pts
@@
 	(wire
 		(pts
-			(xy 96.52 45.72) (xy 93.98 45.72)
-		)
-		(stroke
-			(width 0)
-			(type default)
-		)
-	)
-	(wire
-		(pts
 			(xy 52.07 101.6) (xy 52.07 104.14)
 		)
@@
 	(wire
 		(pts
-			(xy 87.63 45.72) (xy 91.44 45.72)
+			(xy 85.09 45.72) (xy 91.44 45.72)
 		)
 		(stroke
@@
 	(wire
 		(pts
-			(xy 85.09 45.72) (xy 87.63 45.72)
-		)
-		(stroke
-			(width 0)
-			(type default)
-		)
-	)
-	(wire
-		(pts
 			(xy 191.77 97.79) (xy 201.93 97.79)
 		)
@@
 	(wire
 		(pts
-			(xy 87.63 45.72) (xy 87.63 46.99)
-		)
-		(stroke
-			(width 0)
-			(type default)
-		)
-	)
-	(wire
-		(pts
 			(xy 231.14 96.52) (xy 231.14 97.79)
 		)
@@
 	(wire
 		(pts
-			(xy 96.52 45.72) (xy 102.87 45.72)
+			(xy 93.98 45.72) (xy 102.87 45.72)
 		)
 		(stroke
@@
 	(wire
 		(pts
-			(xy 234.95 87.63) (xy 231.14 87.63)
+			(xy 233.68 87.63) (xy 231.14 87.63)
 		)
 		(stroke
@@
 		(pts
 			(xy 39.37 104.14) (xy 52.07 104.14)
-		)
-		(stroke
-			(width 0)
-			(type default)
-		)
-	)
-	(wire
-		(pts
-			(xy 96.52 45.72) (xy 96.52 46.99)
 		)
 		(stroke
@@
 		)
 	)
-	(global_label "72REG"
+	(global_label "AN_IN"
 		(shape input)
-		(at 96.52 46.99 270)
+		(at 133.35 110.49 0)
 		(fields_autoplaced yes)
 		(effects
@@
 				(size 1.27 1.27)
 			)
-			(justify right)
+			(justify left)
 		)
 		(property "Intersheetrefs" "${INTERSHEET_REFS}"
-			(at 96.52 56.0832 90)
-			(effects
-				(font
-					(size 1.27 1.27)
-				)
-				(justify right)
+			(at 141.6572 110.49 0)
+			(effects
+				(font
+					(size 1.27 1.27)
+				)
+				(justify left)
 				(hide yes)
 			)
@@
 	(global_label "BATT+"
 		(shape input)
-		(at 87.63 46.99 270)
-		(fields_autoplaced yes)
-		(effects
-			(font
-				(size 1.27 1.27)
-			)
-			(justify right)
-		)
-		(property "Intersheetrefs" "${INTERSHEET_REFS}"
-			(at 87.63 55.8414 90)
-			(effects
-				(font
-					(size 1.27 1.27)
-				)
-				(justify right)
-				(hide yes)
-			)
-		)
-	)
-	(global_label "BATT+"
-		(shape input)
 		(at 59.69 34.29 0)
 		(fields_autoplaced yes)
@@
 		)
 	)
+	(global_label "Prech"
+		(shape input)
+		(at 93.98 40.64 90)
+		(fields_autoplaced yes)
+		(effects
+			(font
+				(size 1.27 1.27)
+			)
+			(justify left)
+		)
+		(property "Intersheetrefs" "${INTERSHEET_REFS}"
+			(at 93.98 32.2724 90)
+			(effects
+				(font
+					(size 1.27 1.27)
+				)
+				(justify left)
+				(hide yes)
+			)
+		)
+	)
 	(global_label "V+"
 		(shape output)
@@
 		)
 	)
+	(global_label "ErrorVBUS"
+		(shape input)
+		(at 228.6 107.95 0)
+		(fields_autoplaced yes)
+		(effects
+			(font
+				(size 1.27 1.27)
+			)
+			(justify left)
+		)
+		(property "Intersheetrefs" "${INTERSHEET_REFS}"
+			(at 241.1404 107.95 0)
+			(effects
+				(font
+					(size 1.27 1.27)
+				)
+				(justify left)
+				(hide yes)
+			)
+		)
+	)
 	(global_label "V+"
 		(shape output)
@@
 		)
 	)
+	(global_label "BATT"
+		(shape input)
+		(at 91.44 40.64 90)
+		(fields_autoplaced yes)
+		(effects
+			(font
+				(size 1.27 1.27)
+			)
+			(justify left)
+		)
+		(property "Intersheetrefs" "${INTERSHEET_REFS}"
+			(at 91.44 33.361 90)
+			(effects
+				(font
+					(size 1.27 1.27)
+				)
+				(justify left)
+				(hide yes)
+			)
+		)
+	)
+	(global_label "Finish"
+		(shape input)
+		(at 233.68 87.63 0)
+		(fields_autoplaced yes)
+		(effects
+			(font
+				(size 1.27 1.27)
+			)
+			(justify left)
+		)
+		(property "Intersheetrefs" "${INTERSHEET_REFS}"
+			(at 242.2895 87.63 0)
+			(effects
+				(font
+					(size 1.27 1.27)
+				)
+				(justify left)
+				(hide yes)
+			)
+		)
+	)
+	(global_label "Finish"
+		(shape input)
+		(at 133.35 90.17 0)
+		(fields_autoplaced yes)
+		(effects
+			(font
+				(size 1.27 1.27)
+			)
+			(justify left)
+		)
+		(property "Intersheetrefs" "${INTERSHEET_REFS}"
+			(at 141.9595 90.17 0)
+			(effects
+				(font
+					(size 1.27 1.27)
+				)
+				(justify left)
+				(hide yes)
+			)
+		)
+	)
 	(global_label "BATT+"
 		(shape input)
@@
 				(hide yes)
 			)
-		)
-	)
-	(hierarchical_label "Finish"
-		(shape input)
-		(at 234.95 87.63 0)
-		(effects
-			(font
-				(size 1.27 1.27)
-				(thickness 0.1588)
-			)
-			(justify left)
-		)
-	)
-	(hierarchical_label "BATT"
-		(shape input)
-		(at 91.44 40.64 90)
-		(effects
-			(font
-				(size 1.27 1.27)
-				(thickness 0.1588)
-			)
-			(justify left)
-		)
-	)
-	(hierarchical_label "ErrorVBUS"
-		(shape input)
-		(at 228.6 107.95 0)
-		(effects
-			(font
-				(size 1.27 1.27)
-				(thickness 0.1588)
-			)
-			(justify left)
-		)
-	)
-	(hierarchical_label "Finish"
-		(shape input)
-		(at 133.35 90.17 0)
-		(effects
-			(font
-				(size 1.27 1.27)
-				(thickness 0.1588)
-			)
-			(justify left)
-		)
-	)
-	(hierarchical_label "VoltSense"
-		(shape input)
-		(at 133.35 110.49 0)
-		(effects
-			(font
-				(size 1.27 1.27)
-				(thickness 0.1588)
-			)
-			(justify left)
-		)
-	)
-	(hierarchical_label "Prech"
-		(shape input)
-		(at 93.98 40.64 90)
-		(effects
-			(font
-				(size 1.27 1.27)
-				(thickness 0.1588)
-			)
-			(justify left)
 		)
 	)
@@
 			)
 		)
-		(property "Footprint" "Package_SO:SOIC-8-1EP_3.9x4.9mm_P1.27mm_EP2.62x3.51mm"
+		(property "Footprint" "Package_SO:SOIC-8_3.9x4.9mm_P1.27mm"
 			(at 123.19 90.17 0)
 			(effects
@@
 			)
 		)
-		(property "Footprint" "Package_SO:SOIC-8-1EP_3.9x4.9mm_P1.27mm_EP2.62x3.51mm"
+		(property "Footprint" "Package_SO:SOIC-8_3.9x4.9mm_P1.27mm"
 			(at 124.46 110.49 0)
 			(effects
@@
 			)
 		)
-		(property "Footprint" "RELAY180LH:Untitled"
+		(property "Footprint" "RELAY100A:RELAY100A"
 			(at 187.96 124.46 0)
 			(effects
@@
 			)
 		)
-		(property "Footprint" "Package_SO:SOIC-8-1EP_3.9x4.9mm_P1.27mm_EP2.62x3.51mm"
+		(property "Footprint" "Package_SO:SOIC-8_3.9x4.9mm_P1.27mm"
 			(at 123.19 90.17 0)
 			(effects

Commit message: mendekatifix
Parts:
- removed Q3: IRF9540N, Package_TO_SOT_THT:TO-220-3_Vertical, symbol Transistor_FET:IRF9540N
- removed R51, R52: 1K, Resistor_SMD:R_0805_2012Metric_Pad1.20x1.40mm_HandSolder, symbol Device:R
- added FDA117: ~, Custom:FDA117, symbol mosfetDriver:FDA117
- added Q13: IXTY1R6N100D2, Package_TO_SOT_SMD:TO-252-2, symbol Transistor_FET:IPD50R380CE
- added R57: 560, Resistor_SMD:R_0805_2012Metric_Pad1.20x1.40mm_HandSolder, symbol Device:R
- R10: value 500 -> 1k; footprint Package_TO_SOT_THT:TO-247-2_Horizontal_TabDown -> Resistor_THT:R_Axial_DIN0918_L18.0mm_D9.0mm_P30.48mm_Horizontal
- R11: footprint Resistor_SMD:R_2816_7142Metric_Pad3.20x4.45mm_HandSolder -> Resistor_THT:R_Axial_DIN0617_L17.0mm_D6.0mm_P20.32mm_Horizontal
Connections:
- net CTRL+: now also R11.2
- net GND: now also FDA117.1 (in-), FDA117.3 (out+), Q13.3 (S); no longer R11.1
- new net: Q13.2 (D), R11.1
- new net: FDA117.2 (in+), R57.2
- new net: FDA117.4 (out-), Q13.1 (G)
- new net +5V: R57.1
Other:
- moved on the sheet: R10, R11

Commit message: 10nov
Changed lines of the file:
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@@
 		)
 	)
-	(global_label "BATT"
+	(global_label "BATT+"
 		(shape input)
 		(at 91.44 43.18 90)
@@
 		)
 		(property "Intersheetrefs" "${INTERSHEET_REFS}"
-			(at 91.44 35.901 90)
+			(at 91.44 34.3286 90)
 			(effects
 				(font
